File: Episode4/Episode4.kicad_pcb (KiCad board)
At the start: 2 copper layers, 282.6 x 120.7 mm, 205 parts, among them J1 BUS 1, J10 BUS 10, J11 BUS 11, J12 BUS 12, J13 Conn_02x31_Top_Bottom, J14 ATX POWER, J2 BUS 2, J3 BUS 3, J4 BUS 4, J5 BUS 5, J6 BUS 6, J7 BUS 7, J8 BUS 8, J9 BUS 9, SW1 POWER, U1 74HCT14, U2 74HCT74

Commit message: Worked on BOM
Parts:
- added C175: .1µF, Capacitor_SMD:C_0805_2012Metric_Pad1.18x1.45mm_HandSolder, F.Cu at (189.9, 153.8)
- added C176: 470µF, Capacitor_SMD:CP_Elec_8x10.5, F.Cu at (185.8, 209.5)
- added C177: 470µF, Capacitor_SMD:CP_Elec_8x10.5, F.Cu at (185.8, 219.5)
- added C178: 1µF, Capacitor_SMD:C_0805_2012Metric_Pad1.18x1.45mm_HandSolder, F.Cu at (189.9, 156.8)
- added C179: 1µF, Capacitor_SMD:C_0805_2012Metric_Pad1.18x1.45mm_HandSolder, F.Cu at (189.9, 159.8)
- added C180: .1µF, Capacitor_SMD:C_0805_2012Metric_Pad1.18x1.45mm_HandSolder, F.Cu at (189.9, 162.8)
- added C181: .1µF, Capacitor_SMD:C_0805_2012Metric_Pad1.18x1.45mm_HandSolder, F.Cu at (189.9, 165.8)
- added C182: .1µF, Capacitor_SMD:C_0805_2012Metric_Pad1.18x1.45mm_HandSolder, F.Cu at (189.9, 168.8)
- added C183: 220µF, Capacitor_SMD:CP_Elec_10x10.5, F.Cu at (199.8, 179.4)
- added C184: 1µF, Capacitor_SMD:C_0805_2012Metric_Pad1.18x1.45mm_HandSolder, F.Cu at (189.9, 171.8)
- added C185: .1µF, Capacitor_SMD:C_0805_2012Metric_Pad1.18x1.45mm_HandSolder, F.Cu at (189.9, 174.8)
- added C186: .1µF, Capacitor_SMD:C_0805_2012Metric_Pad1.18x1.45mm_HandSolder, F.Cu at (189.9, 177.9)
- added C187: 100µF, Capacitor_SMD:CP_Elec_6.3x5.8, F.Cu at (212.1, 169.6)
- added C188: 1µF, Capacitor_SMD:C_0805_2012Metric_Pad1.18x1.45mm_HandSolder, F.Cu at (189.9, 180.9)
- added C189: .1µF, Capacitor_SMD:C_0805_2012Metric_Pad1.18x1.45mm_HandSolder, F.Cu at (189.9, 183.9)
- added C190: 100µF, Capacitor_SMD:CP_Elec_6.3x5.8, F.Cu at (212.1, 177.8)
- added C191: 1µF, Capacitor_SMD:C_0805_2012Metric_Pad1.18x1.45mm_HandSolder, F.Cu at (189.9, 186.9)
- added C192: .1µF, Capacitor_SMD:C_0805_2012Metric_Pad1.18x1.45mm_HandSolder, F.Cu at (189.9, 189.9)
- added D1: SMBJ5.0A-E3/5B, Diode_SMD:D_SMB, F.Cu at (223.6, 152.0)
- added D2: SMBJ3V3-E3/5B, Diode_SMD:D_SMB, F.Cu at (223.6, 157.6)
- added D3: SMBJ12A-E3/5B, Diode_SMD:D_SMB, F.Cu at (223.6, 163.1)
- added D4: SMBJ12A-E3/5B, Diode_SMD:D_SMB, F.Cu at (223.6, 168.7)
- added D5: SMBJ5.0A-E3/5B, Diode_SMD:D_SMB, F.Cu at (223.6, 174.2)
- added D6: SMBJ3V3-E3/5B, Diode_SMD:D_SMB, F.Cu at (223.6, 179.8)
- added D7: SMBJ12A-E3/5B, Diode_SMD:D_SMB, F.Cu at (223.6, 185.3)
- added D8: SMBJ12A-E3/5B, Diode_SMD:D_SMB, F.Cu at (223.6, 190.9)
- C1, C10, C100, C101, C102, C103, C104, C105, C106, C107, C108, C109, C110, C111, C112, C113, C114, C115, C116, C117, C118, C119, C120, C121, C122, C123, C124, C125, C126, C127, C128, C129, C130, C132, C133, C134, C135, C136, C137, C138, C139, C14, C140, C141, C143, C144, C145, C146, C147, C148, C149, C150, C151, C152, C154, C155, C156, C157, C158, C159, C160, C161, C162, C163, C165, C166, C167, C168, C169, C170, C171, C172, C173, C174, C2, C3, C4, C66, C67, C68, C69, C70, C71, C72, C73, C74, C75, C76, C77, C78, C79, C80, C81, C82, C83, C84, C85, C86, C87, C88, C89, C9, C90, C91, C92, C93, C94, C95, C96, C97, C99: footprint Capacitor_THT:C_Disc_D3.4mm_W2.1mm_P2.50mm -> Capacitor_SMD:C_0805_2012Metric_Pad1.18x1.45mm_HandSolder
- C11, C15, C18: value 100µF -> .1µF; footprint Capacitor_THT:CP_Radial_D6.3mm_P2.50mm -> Capacitor_SMD:C_0805_2012Metric_Pad1.18x1.45mm_HandSolder
- C12: value 1µF -> 470µF; footprint Capacitor_THT:C_Disc_D3.4mm_W2.1mm_P2.50mm -> Capacitor_SMD:CP_Elec_8x10.5
- C13, C142, C164, C17, C20, C7, C8, C98: value .1µF -> 1µF; footprint Capacitor_THT:C_Disc_D3.4mm_W2.1mm_P2.50mm -> Capacitor_SMD:C_0805_2012Metric_Pad1.18x1.45mm_HandSolder
- C131, C153: value 1µF -> .1µF; footprint Capacitor_THT:C_Disc_D3.4mm_W2.1mm_P2.50mm -> Capacitor_SMD:C_0805_2012Metric_Pad1.18x1.45mm_HandSolder
- C16, C19: value 1µF -> 100µF; footprint Capacitor_THT:C_Disc_D3.4mm_W2.1mm_P2.50mm -> Capacitor_SMD:CP_Elec_6.3x5.8
- C21: value 10µF -> .1µF; footprint Capacitor_THT:CP_Radial_D5.0mm_P2.50mm -> Capacitor_SMD:C_0805_2012Metric_Pad1.18x1.45mm_HandSolder
- C22, C23, C24, C25, C26, C27, C28, C29, C30, C31, C32, C33, C34, C35, C36, C37, C38, C39, C40, C41, C42, C43, C44, C45, C46, C47, C48, C49, C50, C51, C52, C53, C54, C55, C56, C57, C58, C59, C60, C61, C62, C63, C64: footprint Capacitor_THT:CP_Radial_D5.0mm_P2.50mm -> Capacitor_SMD:C_1206_3216Metric_Pad1.33x1.80mm_HandSolder
- C5: value 100µF -> 1000µF; footprint Capacitor_THT:CP_Radial_D6.3mm_P2.50mm -> Capacitor_SMD:CP_Elec_10x12.5
- C6: value 1µF -> 1000µF; footprint Capacitor_THT:C_Disc_D3.4mm_W2.1mm_P2.50mm -> Capacitor_SMD:CP_Elec_10x12.5
- C65: value 1µF -> 10µF; footprint Capacitor_THT:C_Disc_D3.4mm_W2.1mm_P2.50mm -> Capacitor_SMD:C_1206_3216Metric_Pad1.33x1.80mm_HandSolder
- R1, R2, R3, R4: footprint Resistor_THT:R_Axial_DIN0207_L6.3mm_D2.5mm_P10.16mm_Horizontal -> Resistor_SMD:R_0805_2012Metric_Pad1.20x1.40mm_HandSolder
- U1, U2: footprint Package_DIP:DIP-14_W7.62mm_Socket_LongPads -> Package_SO:SOIC-14_3.9x8.7mm_P1.27mm
- moved C12 208.5 mm to (185.8, 199.4)
- moved C17 204.3 mm to (151.5, 174.8)
- moved C13 203.9 mm to (151.5, 165.8)
- moved C14 203.5 mm to (151.5, 168.8)
- moved C11 195.6 mm to (151.5, 162.8), turned to 0 degrees
- moved C15 195.0 mm to (151.5, 171.8), turned to 0 degrees
- moved C20 187.9 mm to (151.5, 180.9)
- moved C7 167.5 mm to (151.5, 150.8)
- moved C8 167.2 mm to (151.5, 153.8)
- moved C9 167.0 mm to (151.5, 156.8)
- moved C10 166.8 mm to (151.5, 159.8)
- moved C18 163.6 mm to (151.5, 177.9), turned to 0 degrees
- moved C16 154.3 mm to (212.1, 153.3)
- moved C6 134.1 mm to (199.8, 167.3)
- moved C19 127.3 mm to (212.1, 161.5)
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Connections:
- C109 pad 1: +5V -> +3V3
- C11 pad 1: +3V3 -> +5V
- C131 pad 1: +12V -> +5V
- C15 pad 1: +12V -> +3V3
- C153 pad 1: -12V -> +12V
- C18 pad 1: GND -> +12V
- C18 pad 2: -12V -> GND
- C19 pad 1: -12V -> GND
- C19 pad 2: GND -> -12V
- C21 pad 1: +5V -> -12V
- C43 pad 1: +3V3 -> +5V
- C54 pad 1: +12V -> +3V3
- C60 pad 1: GND -> +12V
- C60 pad 2: -12V -> GND
- C65 pad 1: +5V -> GND
- C65 pad 2: GND -> -12V
- C87 pad 1: +3V3 -> +5V
Routing:
- net Net-(SW1-A): track 1.16 -> 0.00 mm
Other:
- board size 282.6 x 120.7 mm -> 282.6 x 114.3 mm

Commit message: Changed bus from 62 to 72 pins
Parts:
- removed the C3 at (230.2, 167.1)
- removed the C4 at (230.2, 170.2)
- removed the J14 at (302.2, 67.5)
- added C174: .1µF, Capacitor_SMD:C_0805_2012Metric_Pad1.18x1.45mm_HandSolder, F.Cu at (426.4, 59.1)
- added C175: .1µF, Capacitor_SMD:C_0805_2012Metric_Pad1.18x1.45mm_HandSolder, F.Cu at (426.4, 62.1)
- added J8: ATX POWER, MicroHobbyist:ATX_PSU_CONN, F.Cu at (394.8, 69.4)
- C10: renamed from C12; value 470µF -> 100µF; footprint Capacitor_SMD:CP_Elec_8x10.5 -> Capacitor_SMD:CP_Elec_6.3x7.7
- C14: renamed from C16; footprint Capacitor_SMD:CP_Elec_6.3x5.8 -> Capacitor_SMD:CP_Elec_6.3x7.7
- C17: renamed from C19; footprint Capacitor_SMD:CP_Elec_6.3x5.8 -> Capacitor_SMD:CP_Elec_6.3x7.7
- C176, C177: value 470µF -> 100µF; footprint Capacitor_SMD:CP_Elec_8x10.5 -> Capacitor_SMD:CP_Elec_6.3x7.7
- C183: value 220µF -> 100µF; footprint Capacitor_SMD:CP_Elec_10x10.5 -> Capacitor_SMD:CP_Elec_6.3x7.7
- C187, C190: footprint Capacitor_SMD:CP_Elec_6.3x5.8 -> Capacitor_SMD:CP_Elec_6.3x7.7
- C20: renamed from C22; footprint Capacitor_SMD:C_1206_3216Metric_Pad1.33x1.80mm_HandSolder -> Capacitor_SMD:CP_Elec_4x5.8
- C21: renamed from C23; footprint Capacitor_SMD:C_1206_3216Metric_Pad1.33x1.80mm_HandSolder -> Capacitor_SMD:CP_Elec_4x5.8
- C22: renamed from C24; footprint Capacitor_SMD:C_1206_3216Metric_Pad1.33x1.80mm_HandSolder -> Capacitor_SMD:CP_Elec_4x5.8
- C23: renamed from C25; footprint Capacitor_SMD:C_1206_3216Metric_Pad1.33x1.80mm_HandSolder -> Capacitor_SMD:CP_Elec_4x5.8
- C24: renamed from C26; footprint Capacitor_SMD:C_1206_3216Metric_Pad1.33x1.80mm_HandSolder -> Capacitor_SMD:CP_Elec_4x5.8
- C25: renamed from C27; footprint Capacitor_SMD:C_1206_3216Metric_Pad1.33x1.80mm_HandSolder -> Capacitor_SMD:CP_Elec_4x5.8
- C26: renamed from C28; footprint Capacitor_SMD:C_1206_3216Metric_Pad1.33x1.80mm_HandSolder -> Capacitor_SMD:CP_Elec_4x5.8
- C27: renamed from C29; footprint Capacitor_SMD:C_1206_3216Metric_Pad1.33x1.80mm_HandSolder -> Capacitor_SMD:CP_Elec_4x5.8
- C28: renamed from C30; footprint Capacitor_SMD:C_1206_3216Metric_Pad1.33x1.80mm_HandSolder -> Capacitor_SMD:CP_Elec_4x5.8
- C29: renamed from C31; footprint Capacitor_SMD:C_1206_3216Metric_Pad1.33x1.80mm_HandSolder -> Capacitor_SMD:CP_Elec_4x5.8
- C3: renamed from C5; value 1000µF -> 100µF; footprint Capacitor_SMD:CP_Elec_10x12.5 -> Capacitor_SMD:CP_Elec_6.3x7.7
- C30: renamed from C32; footprint Capacitor_SMD:C_1206_3216Metric_Pad1.33x1.80mm_HandSolder -> Capacitor_SMD:CP_Elec_4x5.8
- C31: renamed from C33; footprint Capacitor_SMD:C_1206_3216Metric_Pad1.33x1.80mm_HandSolder -> Capacitor_SMD:CP_Elec_4x5.8
- C32: renamed from C34; footprint Capacitor_SMD:C_1206_3216Metric_Pad1.33x1.80mm_HandSolder -> Capacitor_SMD:CP_Elec_4x5.8
- C33: renamed from C35; footprint Capacitor_SMD:C_1206_3216Metric_Pad1.33x1.80mm_HandSolder -> Capacitor_SMD:CP_Elec_4x5.8
- C34: renamed from C36; footprint Capacitor_SMD:C_1206_3216Metric_Pad1.33x1.80mm_HandSolder -> Capacitor_SMD:CP_Elec_4x5.8
- C35: renamed from C37; footprint Capacitor_SMD:C_1206_3216Metric_Pad1.33x1.80mm_HandSolder -> Capacitor_SMD:CP_Elec_4x5.8
- C36: renamed from C38; footprint Capacitor_SMD:C_1206_3216Metric_Pad1.33x1.80mm_HandSolder -> Capacitor_SMD:CP_Elec_4x5.8
- C37: renamed from C39; footprint Capacitor_SMD:C_1206_3216Metric_Pad1.33x1.80mm_HandSolder -> Capacitor_SMD:CP_Elec_4x5.8
- C38: renamed from C40; footprint Capacitor_SMD:C_1206_3216Metric_Pad1.33x1.80mm_HandSolder -> Capacitor_SMD:CP_Elec_4x5.8
- C39: renamed from C41; footprint Capacitor_SMD:C_1206_3216Metric_Pad1.33x1.80mm_HandSolder -> Capacitor_SMD:CP_Elec_4x5.8
- C4: renamed from C6; value 1000µF -> 100µF; footprint Capacitor_SMD:CP_Elec_10x12.5 -> Capacitor_SMD:CP_Elec_6.3x7.7
- C40: renamed from C42; footprint Capacitor_SMD:C_1206_3216Metric_Pad1.33x1.80mm_HandSolder -> Capacitor_SMD:CP_Elec_4x5.8
- C41: renamed from C43; footprint Capacitor_SMD:C_1206_3216Metric_Pad1.33x1.80mm_HandSolder -> Capacitor_SMD:CP_Elec_4x5.8
- C42: renamed from C44; footprint Capacitor_SMD:C_1206_3216Metric_Pad1.33x1.80mm_HandSolder -> Capacitor_SMD:CP_Elec_4x5.8
- C43: renamed from C45; footprint Capacitor_SMD:C_1206_3216Metric_Pad1.33x1.80mm_HandSolder -> Capacitor_SMD:CP_Elec_4x5.8
- C44: renamed from C46; footprint Capacitor_SMD:C_1206_3216Metric_Pad1.33x1.80mm_HandSolder -> Capacitor_SMD:CP_Elec_4x5.8
- C45: renamed from C47; footprint Capacitor_SMD:C_1206_3216Metric_Pad1.33x1.80mm_HandSolder -> Capacitor_SMD:CP_Elec_4x5.8
- C46: renamed from C48; footprint Capacitor_SMD:C_1206_3216Metric_Pad1.33x1.80mm_HandSolder -> Capacitor_SMD:CP_Elec_4x5.8
- C47: renamed from C49; footprint Capacitor_SMD:C_1206_3216Metric_Pad1.33x1.80mm_HandSolder -> Capacitor_SMD:CP_Elec_4x5.8
- C48: renamed from C50; footprint Capacitor_SMD:C_1206_3216Metric_Pad1.33x1.80mm_HandSolder -> Capacitor_SMD:CP_Elec_4x5.8
- C49: renamed from C51; footprint Capacitor_SMD:C_1206_3216Metric_Pad1.33x1.80mm_HandSolder -> Capacitor_SMD:CP_Elec_4x5.8
- C50: renamed from C52; footprint Capacitor_SMD:C_1206_3216Metric_Pad1.33x1.80mm_HandSolder -> Capacitor_SMD:CP_Elec_4x5.8
- C51: renamed from C53; footprint Capacitor_SMD:C_1206_3216Metric_Pad1.33x1.80mm_HandSolder -> Capacitor_SMD:CP_Elec_4x5.8
- C52: renamed from C54; footprint Capacitor_SMD:C_1206_3216Metric_Pad1.33x1.80mm_HandSolder -> Capacitor_SMD:CP_Elec_4x5.8
- C53: renamed from C55; footprint Capacitor_SMD:C_1206_3216Metric_Pad1.33x1.80mm_HandSolder -> Capacitor_SMD:CP_Elec_4x5.8
- C54: renamed from C56; footprint Capacitor_SMD:C_1206_3216Metric_Pad1.33x1.80mm_HandSolder -> Capacitor_SMD:CP_Elec_4x5.8
- C55: renamed from C57; footprint Capacitor_SMD:C_1206_3216Metric_Pad1.33x1.80mm_HandSolder -> Capacitor_SMD:CP_Elec_4x5.8
- C56: renamed from C58; footprint Capacitor_SMD:C_1206_3216Metric_Pad1.33x1.80mm_HandSolder -> Capacitor_SMD:CP_Elec_4x5.8
- C57: renamed from C59; footprint Capacitor_SMD:C_1206_3216Metric_Pad1.33x1.80mm_HandSolder -> Capacitor_SMD:CP_Elec_4x5.8
- C58: renamed from C60; footprint Capacitor_SMD:C_1206_3216Metric_Pad1.33x1.80mm_HandSolder -> Capacitor_SMD:CP_Elec_4x5.8
- C59: renamed from C61; footprint Capacitor_SMD:C_1206_3216Metric_Pad1.33x1.80mm_HandSolder -> Capacitor_SMD:CP_Elec_4x5.8
- C60: renamed from C62; footprint Capacitor_SMD:C_1206_3216Metric_Pad1.33x1.80mm_HandSolder -> Capacitor_SMD:CP_Elec_4x5.8
- C61: renamed from C63; footprint Capacitor_SMD:C_1206_3216Metric_Pad1.33x1.80mm_HandSolder -> Capacitor_SMD:CP_Elec_4x5.8
- C62: renamed from C64; footprint Capacitor_SMD:C_1206_3216Metric_Pad1.33x1.80mm_HandSolder -> Capacitor_SMD:CP_Elec_4x5.8
- C63: renamed from C65; footprint Capacitor_SMD:C_1206_3216Metric_Pad1.33x1.80mm_HandSolder -> Capacitor_SMD:CP_Elec_4x5.8
- D1, D5: value SMBJ5.0A-E3/5B -> TVS 5V
- D2, D6: value SMBJ3V3-E3/5B -> TVS 3V3
- D3, D4, D7, D8: value SMBJ12A-E3/5B -> TVS 12V
- J1: value BUS 1 -> CARD; footprint MicroHobbyist:ISA_Connector -> MicroHobbyist:72-pin CE connector
- J10: renamed from J8; value BUS 8 -> CARD; footprint MicroHobbyist:ISA_Connector -> MicroHobbyist:72-pin CE connector
- J11: renamed from J9; value BUS 9 -> CARD; footprint MicroHobbyist:ISA_Connector -> MicroHobbyist:72-pin CE connector
- J12: renamed from J10; value BUS 10 -> CARD; footprint MicroHobbyist:ISA_Connector -> MicroHobbyist:72-pin CE connector
- J13: renamed from J11; value BUS 11 -> CARD; footprint MicroHobbyist:ISA_Connector -> MicroHobbyist:72-pin CE connector
- J14: renamed from J12; value BUS 12 -> CARD; footprint MicroHobbyist:ISA_Connector -> MicroHobbyist:72-pin CE connector
- J2: value BUS 2 -> CARD; footprint MicroHobbyist:ISA_Connector -> MicroHobbyist:72-pin CE connector
- J3: value BUS 3 -> CARD; footprint MicroHobbyist:ISA_Connector -> MicroHobbyist:72-pin CE connector
- J4: value BUS 4 -> CARD; footprint MicroHobbyist:ISA_Connector -> MicroHobbyist:72-pin CE connector
- J5: value BUS 5 -> CARD; footprint MicroHobbyist:ISA_Connector -> MicroHobbyist:72-pin CE connector
- J6: value BUS 6 -> CARD; footprint MicroHobbyist:ISA_Connector -> MicroHobbyist:72-pin CE connector
- J7: renamed from J13; value Conn_02x31_Top_Bottom -> BB Con; footprint Connector_PinSocket_2.54mm:PinSocket_2x31_P2.54mm_Vertical -> Connector_PinSocket_2.54mm:PinSocket_2x36_P2.54mm_Vertical
- J9: renamed from J7; value BUS 7 -> CARD; footprint MicroHobbyist:ISA_Connector -> MicroHobbyist:72-pin CE connector
- R3: value 20K -> 330
- R4: value 220 -> 20K
- SW1: footprint MicroHobbyist:Pushbutton_12mm_LED -> MicroHobbyist:TS2912121G300D
- moved H6 355.2 mm to (385.4, 76.2)
- moved H1 348.6 mm to (376.9, 76.2)
- moved H10 301.9 mm to (385.4, 110.4)
- moved H2 287.1 mm to (376.9, 84.8)
- moved H9 240.9 mm to (385.4, 101.9)
- moved H3 225.5 mm to (376.9, 93.3)
- moved C177 220.1 mm to (301.6, 32.4)
- moved C176 217.6 mm to (60.3, 31.8)
- moved C178 209.5 mm to (-9.93, 94.0)
- moved C179 209.5 mm to (-9.93, 97.0)
- moved C180 209.5 mm to (-9.93, 100.0)
- moved C181 209.5 mm to (-9.93, 103.1)
- moved C182 209.5 mm to (-9.93, 106.1)
- moved C184 209.5 mm to (-9.93, 109.1)
- moved C185 209.5 mm to (-9.93, 112.1)
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- renumbered C102 to C100, C103 to C101, C104 to C102, C105 to C103, C106 to C104, C107 to C105, C108 to C106, C109 to C107, C110 to C108, C111 to C109, C13 to C11, C112 to C110, C113 to C111, C114 to C112, C115 to C113, C116 to C114, C117 to C115, C118 to C116, C119 to C117, C120 to C118, C121 to C119, C14 to C12, C122 to C120, C123 to C121, C124 to C122, C125 to C123, C126 to C124, C127 to C125, C128 to C126, C129 to C127, C130 to C128, C131 to C129, C15 to C13, C132 to C130, C133 to C131, C134 to C132, C135 to C133, C136 to C134, C137 to C135, C138 to C136, C139 to C137, C140 to C138, C141 to C139, C142 to C140, C143 to C141, C144 to C142, C145 to C143, C146 to C144, C147 to C145, C148 to C146, C149 to C147, C150 to C148, C151 to C149, C17 to C15, C152 to C150, C153 to C151, C154 to C152, C155 to C153, C156 to C154, C157 to C155, C158 to C156, C159 to C157, C160 to C158, C161 to C159, C18 to C16, C162 to C160, C163 to C161, C164 to C162, C165 to C163, C166 to C164, C167 to C165, C168 to C166, C169 to C167, C170 to C168, C171 to C169, C172 to C170, C173 to C171, C174 to C172, C175 to C173, C20 to C18, C21 to C19, C7 to C5, C8 to C6, C66 to C64, C67 to C65, C68 to C66, C69 to C67, C70 to C68, C71 to C69, C9 to C7, C72 to C70, C73 to C71, C74 to C72, C75 to C73, C76 to C74, C77 to C75, C78 to C76, C79 to C77, C80 to C78, C81 to C79, C10 to C8, C82 to C80, C83 to C81, C84 to C82, C85 to C83, C86 to C84, C87 to C85, C88 to C86, C89 to C87, C90 to C88, C91 to C89, C11 to C9, C92 to C90, C93 to C91, C94 to C92, C95 to C93, C96 to C94, C97 to C95, C98 to C96, C99 to C97, C100 to C98, C101 to C99
Connections:
- J1 pad 1: /A0 -> +5V
- J1 pad 10: /A9 -> /~{RD}
- J1 pad 11: /A10 -> /A3
- J1 pad 12: /A11 -> /~{WR}
- J1 pad 13: /A12 -> /A4
- J1 pad 14: /A13 -> /R/~{W}
- J1 pad 15: /A14 -> /A5
- J1 pad 16: /A15 -> /~{CART_{en}}
- J1 pad 17: GND -> /A6
- J1 pad 18: -12V -> /CLK1
- J1 pad 19: +12V -> /A7
- J1 pad 2: /A1 -> +5V
- J1 pad 20: GND -> /CLK2
- J1 pad 21: +3V3 -> GND
- J1 pad 22: +3V3 -> GND
- J1 pad 23: GND -> /A8
- J1 pad 24: /D0 -> /RESET
- J1 pad 25: /D1 -> /A9
- J1 pad 26: /D2 -> /~{MREQ}
- J1 pad 27: /D3 -> /A10
- J1 pad 28: /D4 -> /~{IORQ}
- J1 pad 29: /D5 -> /A11
- J1 pad 3: /A2 -> GND
- J1 pad 30: /D6 -> /~{CBLK}
- J1 pad 31: /D7 -> /A12
- J1 pad 32: GND -> /~{BREQ}
- J1 pad 33: +5V -> /A13
- J1 pad 34: +5V -> /~{HALT}
- J1 pad 35: GND -> /A14
- J1 pad 36: /E -> /~{MRDY}
- J1 pad 37: /Q -> /A15
- J1 pad 38: /~{VMA} -> /~{ROM_{cs}}
- J1 pad 39: GND -> /~{MMU_{en}}
- J1 pad 4: /A3 -> GND
- J1 pad 40: /R/~{W} -> /~{RAM_{oe}}
- J1 pad 41: /~{RD} -> GND
- J1 pad 42: /~{WR} -> GND
- J1 pad 43: /~{RAM_{oe}} -> +3V3
- J1 pad 44: GND -> +3V3
- J1 pad 45: /~{CBLK} -> GND
- J1 pad 46: /~{IORQ} -> GND
- J1 pad 47: /~{MREQ} -> +12V
- J1 pad 48: /~{HALT} -> /BA
- J1 pad 49: /~{MRDY} -> -12V
- J1 pad 5: /A4 -> /A0
- J1 pad 50: /~{BREQ} -> /BS
- J1 pad 52: /BA -> GND
- J1 pad 53: /BS -> /D0
- J1 pad 54: /SPARE -> /USR1
- J1 pad 55: /~{RESET} -> /D1
- J1 pad 56: /~{NMI} -> /USR2
- J1 pad 57: /~{IRQ} -> /D2
- J1 pad 58: /~{FIRQ} -> /USR3
- J1 pad 59: GND -> /D3
- J1 pad 6: /A5 -> /Q
- J1 pad 60: +5V -> /USR4
- J1 pad 61: +5V -> /D4
- J1 pad 62: GND -> /~{RESET}
- J1 pad 7: /A6 -> /A1
- J1 pad 8: /A7 -> /E
- J1 pad 9: /A8 -> /A2
- J10 pad 1: /A0 -> +5V
- J10 pad 10: /A9 -> /~{RD}
- J10 pad 11: /A10 -> /A3
- J10 pad 12: /A11 -> /~{WR}
- J10 pad 13: /A12 -> /A4
- J10 pad 14: /A13 -> /R/~{W}
- J10 pad 15: /A14 -> /A5
- J10 pad 16: /A15 -> /~{CART_{en}}
- J10 pad 17: GND -> /A6
- J10 pad 18: -12V -> /CLK1
- J10 pad 19: +12V -> /A7
- J10 pad 2: /A1 -> +5V
- J10 pad 20: GND -> /CLK2
- J10 pad 21: +3V3 -> GND
- J10 pad 22: +3V3 -> GND
- J10 pad 23: GND -> /A8
- J10 pad 24: /D0 -> /RESET
- J10 pad 25: /D1 -> /A9
- J10 pad 26: /D2 -> /~{MREQ}
- J10 pad 27: /D3 -> /A10
- J10 pad 28: /D4 -> /~{IORQ}
- J10 pad 29: /D5 -> /A11
- J10 pad 3: /A2 -> GND
- J10 pad 30: /D6 -> /~{CBLK}
- J10 pad 31: /D7 -> /A12
- J10 pad 32: GND -> /~{BREQ}
- J10 pad 33: +5V -> /A13
- J10 pad 34: +5V -> /~{HALT}
- J10 pad 35: GND -> /A14
- J10 pad 36: /E -> /~{MRDY}
- J10 pad 37: /Q -> /A15
- J10 pad 38: /~{VMA} -> /~{ROM_{cs}}
- J10 pad 39: GND -> /~{MMU_{en}}
- J10 pad 4: /A3 -> GND
- J10 pad 40: /R/~{W} -> /~{RAM_{oe}}
- J10 pad 41: /~{RD} -> GND
- J10 pad 42: /~{WR} -> GND
- J10 pad 43: /~{RAM_{oe}} -> +3V3
- J10 pad 44: GND -> +3V3
- J10 pad 45: /~{CBLK} -> GND
- J10 pad 46: /~{IORQ} -> GND
- J10 pad 47: /~{MREQ} -> +12V
- J10 pad 48: /~{HALT} -> /BA
- J10 pad 49: /~{MRDY} -> -12V
- J10 pad 5: /A4 -> /A0
- J10 pad 50: /~{BREQ} -> /BS
- J10 pad 52: /BA -> GND
- J10 pad 53: /BS -> /D0
- J10 pad 54: /SPARE -> /USR1
- J10 pad 55: /~{RESET} -> /D1
- J10 pad 56: /~{NMI} -> /USR2
- J10 pad 57: /~{IRQ} -> /D2
- J10 pad 58: /~{FIRQ} -> /USR3
- J10 pad 59: GND -> /D3
- J10 pad 6: /A5 -> /Q
- J10 pad 60: +5V -> /USR4
- J10 pad 61: +5V -> /D4
- J10 pad 62: GND -> /~{RESET}
- J10 pad 7: /A6 -> /A1
- J10 pad 8: /A7 -> /E
- J10 pad 9: /A8 -> /A2
- J11 pad 1: /A0 -> +5V
- J11 pad 10: /A9 -> /~{RD}
- J11 pad 11: /A10 -> /A3
- J11 pad 12: /A11 -> /~{WR}
- J11 pad 13: /A12 -> /A4
- J11 pad 14: /A13 -> /R/~{W}
- J11 pad 15: /A14 -> /A5
- J11 pad 16: /A15 -> /~{CART_{en}}
- J11 pad 17: GND -> /A6
- J11 pad 18: -12V -> /CLK1
- J11 pad 19: +12V -> /A7
- J11 pad 2: /A1 -> +5V
- J11 pad 20: GND -> /CLK2
- J11 pad 21: +3V3 -> GND
- J11 pad 22: +3V3 -> GND
- J11 pad 23: GND -> /A8
- J11 pad 24: /D0 -> /RESET
- J11 pad 25: /D1 -> /A9
- J11 pad 26: /D2 -> /~{MREQ}
- J11 pad 27: /D3 -> /A10
- J11 pad 28: /D4 -> /~{IORQ}
- J11 pad 29: /D5 -> /A11
- J11 pad 3: /A2 -> GND
- J11 pad 30: /D6 -> /~{CBLK}
- J11 pad 31: /D7 -> /A12
- J11 pad 32: GND -> /~{BREQ}
- J11 pad 33: +5V -> /A13
- J11 pad 34: +5V -> /~{HALT}
- J11 pad 35: GND -> /A14
- J11 pad 36: /E -> /~{MRDY}
- J11 pad 37: /Q -> /A15
- J11 pad 38: /~{VMA} -> /~{ROM_{cs}}
- J11 pad 39: GND -> /~{MMU_{en}}
- J11 pad 4: /A3 -> GND
- J11 pad 40: /R/~{W} -> /~{RAM_{oe}}
- J11 pad 41: /~{RD} -> GND
- J11 pad 42: /~{WR} -> GND
- J11 pad 43: /~{RAM_{oe}} -> +3V3
- J11 pad 44: GND -> +3V3
- J11 pad 45: /~{CBLK} -> GND
- J11 pad 46: /~{IORQ} -> GND
- J11 pad 47: /~{MREQ} -> +12V
- J11 pad 48: /~{HALT} -> /BA
- J11 pad 49: /~{MRDY} -> -12V
- J11 pad 5: /A4 -> /A0
- J11 pad 50: /~{BREQ} -> /BS
- J11 pad 52: /BA -> GND
- J11 pad 53: /BS -> /D0
- J11 pad 54: /SPARE -> /USR1
- J11 pad 55: /~{RESET} -> /D1
- J11 pad 56: /~{NMI} -> /USR2
- J11 pad 57: /~{IRQ} -> /D2
- J11 pad 58: /~{FIRQ} -> /USR3
- J11 pad 59: GND -> /D3
- J11 pad 6: /A5 -> /Q
- J11 pad 60: +5V -> /USR4
- J11 pad 61: +5V -> /D4
- J11 pad 62: GND -> /~{RESET}
- J11 pad 7: /A6 -> /A1
- J11 pad 8: /A7 -> /E
- J11 pad 9: /A8 -> /A2
- J12 pad 1: /A0 -> +5V
- J12 pad 10: /A9 -> /~{RD}
- J12 pad 11: /A10 -> /A3
- J12 pad 12: /A11 -> /~{WR}
- J12 pad 13: /A12 -> /A4
- J12 pad 14: /A13 -> /R/~{W}
- J12 pad 15: /A14 -> /A5
- J12 pad 16: /A15 -> /~{CART_{en}}
- J12 pad 17: GND -> /A6
- J12 pad 18: -12V -> /CLK1
- J12 pad 19: +12V -> /A7
- J12 pad 2: /A1 -> +5V
- J12 pad 20: GND -> /CLK2
- J12 pad 21: +3V3 -> GND
- J12 pad 22: +3V3 -> GND
- J12 pad 23: GND -> /A8
- J12 pad 24: /D0 -> /RESET
- J12 pad 25: /D1 -> /A9
- J12 pad 26: /D2 -> /~{MREQ}
- J12 pad 27: /D3 -> /A10
- J12 pad 28: /D4 -> /~{IORQ}
- J12 pad 29: /D5 -> /A11
- J12 pad 3: /A2 -> GND
- J12 pad 30: /D6 -> /~{CBLK}
- J12 pad 31: /D7 -> /A12
- J12 pad 32: GND -> /~{BREQ}
- J12 pad 33: +5V -> /A13
- J12 pad 34: +5V -> /~{HALT}
- J12 pad 35: GND -> /A14
- J12 pad 36: /E -> /~{MRDY}
- J12 pad 37: /Q -> /A15
- J12 pad 38: /~{VMA} -> /~{ROM_{cs}}
- J12 pad 39: GND -> /~{MMU_{en}}
- J12 pad 4: /A3 -> GND
- J12 pad 40: /R/~{W} -> /~{RAM_{oe}}
- J12 pad 41: /~{RD} -> GND
- J12 pad 42: /~{WR} -> GND
- J12 pad 43: /~{RAM_{oe}} -> +3V3
- J12 pad 44: GND -> +3V3
- J12 pad 45: /~{CBLK} -> GND
- J12 pad 46: /~{IORQ} -> GND
- J12 pad 47: /~{MREQ} -> +12V
- J12 pad 48: /~{HALT} -> /BA
- J12 pad 49: /~{MRDY} -> -12V
- J12 pad 5: /A4 -> /A0
- J12 pad 50: /~{BREQ} -> /BS
- J12 pad 52: /BA -> GND
- J12 pad 53: /BS -> /D0
- J12 pad 54: /SPARE -> /USR1
- J12 pad 55: /~{RESET} -> /D1
- J12 pad 56: /~{NMI} -> /USR2
- J12 pad 57: /~{IRQ} -> /D2
- J12 pad 58: /~{FIRQ} -> /USR3
- J12 pad 59: GND -> /D3
- J12 pad 6: /A5 -> /Q
- J12 pad 60: +5V -> /USR4
- J12 pad 61: +5V -> /D4
- J12 pad 62: GND -> /~{RESET}
- J12 pad 7: /A6 -> /A1
- J12 pad 8: /A7 -> /E
- J12 pad 9: /A8 -> /A2
- J13 pad 1: /A0 -> +5V
- J13 pad 10: /A9 -> /~{RD}
- J13 pad 11: /A10 -> /A3
- J13 pad 12: /A11 -> /~{WR}
- J13 pad 13: /A12 -> /A4
- J13 pad 14: /A13 -> /R/~{W}
- J13 pad 15: /A14 -> /A5
- J13 pad 16: /A15 -> /~{CART_{en}}
- J13 pad 17: GND -> /A6
- J13 pad 18: -12V -> /CLK1
- J13 pad 19: +12V -> /A7
- J13 pad 2: /A1 -> +5V
- J13 pad 20: GND -> /CLK2
- J13 pad 21: +3V3 -> GND
- J13 pad 22: +3V3 -> GND
- J13 pad 23: GND -> /A8
- J13 pad 24: /D0 -> /RESET
- J13 pad 25: /D1 -> /A9
- J13 pad 26: /D2 -> /~{MREQ}
- J13 pad 27: /D3 -> /A10
- J13 pad 28: /D4 -> /~{IORQ}
- J13 pad 29: /D5 -> /A11
- J13 pad 3: /A2 -> GND
- J13 pad 30: /D6 -> /~{CBLK}
- J13 pad 31: /D7 -> /A12
- J13 pad 32: GND -> /~{BREQ}
- J13 pad 33: +5V -> /A13
- J13 pad 34: +5V -> /~{HALT}
- J13 pad 35: GND -> /A14
- J13 pad 36: /E -> /~{MRDY}
- J13 pad 37: /Q -> /A15
- J13 pad 38: /~{VMA} -> /~{ROM_{cs}}
- J13 pad 39: GND -> /~{MMU_{en}}
- J13 pad 4: /A3 -> GND
- J13 pad 40: /R/~{W} -> /~{RAM_{oe}}
- J13 pad 41: /~{RD} -> GND
- J13 pad 42: /~{WR} -> GND
- J13 pad 43: /~{RAM_{oe}} -> +3V3
- J13 pad 44: GND -> +3V3
- J13 pad 45: /~{CBLK} -> GND
- J13 pad 46: /~{IORQ} -> GND
- J13 pad 47: /~{MREQ} -> +12V
- J13 pad 48: /~{HALT} -> /BA
- J13 pad 49: /~{MRDY} -> -12V
- J13 pad 5: /A4 -> /A0
- J13 pad 50: /~{BREQ} -> /BS
- J13 pad 52: /BA -> GND
- J13 pad 53: /BS -> /D0
- J13 pad 54: /SPARE -> /USR1
- J13 pad 55: /~{RESET} -> /D1
- J13 pad 56: /~{NMI} -> /USR2
- J13 pad 57: /~{IRQ} -> /D2
- J13 pad 58: /~{FIRQ} -> /USR3
- J13 pad 59: GND -> /D3
- J13 pad 6: /A5 -> /Q
- J13 pad 60: +5V -> /USR4
- J13 pad 61: +5V -> /D4
- J13 pad 62: GND -> /~{RESET}
- J13 pad 7: /A6 -> /A1
- J13 pad 8: /A7 -> /E
- J13 pad 9: /A8 -> /A2
- J14 pad 1: /A0 -> +5V
- J14 pad 10: /A9 -> /~{RD}
- J14 pad 11: /A10 -> /A3
- J14 pad 12: /A11 -> /~{WR}
- J14 pad 13: /A12 -> /A4
- J14 pad 14: /A13 -> /R/~{W}
- J14 pad 15: /A14 -> /A5
- J14 pad 16: /A15 -> /~{CART_{en}}
- J14 pad 17: GND -> /A6
- J14 pad 18: -12V -> /CLK1
- J14 pad 19: +12V -> /A7
- J14 pad 2: /A1 -> +5V
- J14 pad 20: GND -> /CLK2
- J14 pad 21: +3V3 -> GND
- J14 pad 22: +3V3 -> GND
- J14 pad 23: GND -> /A8
- J14 pad 24: /D0 -> /RESET
- J14 pad 25: /D1 -> /A9
- J14 pad 26: /D2 -> /~{MREQ}
- J14 pad 27: /D3 -> /A10
- J14 pad 28: /D4 -> /~{IORQ}
- J14 pad 29: /D5 -> /A11
- J14 pad 3: /A2 -> GND
- J14 pad 30: /D6 -> /~{CBLK}
- J14 pad 31: /D7 -> /A12
- J14 pad 32: GND -> /~{BREQ}
- J14 pad 33: +5V -> /A13
- J14 pad 34: +5V -> /~{HALT}
- J14 pad 35: GND -> /A14
- J14 pad 36: /E -> /~{MRDY}
- J14 pad 37: /Q -> /A15
- J14 pad 38: /~{VMA} -> /~{ROM_{cs}}
- J14 pad 39: GND -> /~{MMU_{en}}
- J14 pad 4: /A3 -> GND
- J14 pad 40: /R/~{W} -> /~{RAM_{oe}}
- J14 pad 41: /~{RD} -> GND
- J14 pad 42: /~{WR} -> GND
- J14 pad 43: /~{RAM_{oe}} -> +3V3
- J14 pad 44: GND -> +3V3
- J14 pad 45: /~{CBLK} -> GND
- J14 pad 46: /~{IORQ} -> GND
- J14 pad 47: /~{MREQ} -> +12V
- J14 pad 48: /~{HALT} -> /BA
- J14 pad 49: /~{MRDY} -> -12V
- J14 pad 5: /A4 -> /A0
- J14 pad 50: /~{BREQ} -> /BS
- J14 pad 52: /BA -> GND
- J14 pad 53: /BS -> /D0
- J14 pad 54: /SPARE -> /USR1
- J14 pad 55: /~{RESET} -> /D1
- J14 pad 56: /~{NMI} -> /USR2
- J14 pad 57: /~{IRQ} -> /D2
- J14 pad 58: /~{FIRQ} -> /USR3
- J14 pad 59: GND -> /D3
- J14 pad 6: /A5 -> /Q
- J14 pad 60: +5V -> /USR4
- J14 pad 61: +5V -> /D4
- J14 pad 62: GND -> /~{RESET}
- J14 pad 7: /A6 -> /A1
- J14 pad 8: /A7 -> /E
- J14 pad 9: /A8 -> /A2
- J2 pad 1: /A0 -> +5V
- J2 pad 10: /A9 -> /~{RD}
- J2 pad 11: /A10 -> /A3
- J2 pad 12: /A11 -> /~{WR}
- J2 pad 13: /A12 -> /A4
- J2 pad 14: /A13 -> /R/~{W}
- J2 pad 15: /A14 -> /A5
- J2 pad 16: /A15 -> /~{CART_{en}}
- J2 pad 17: GND -> /A6
- J2 pad 18: -12V -> /CLK1
- J2 pad 19: +12V -> /A7
- J2 pad 2: /A1 -> +5V
- J2 pad 20: GND -> /CLK2
- J2 pad 21: +3V3 -> GND
- J2 pad 22: +3V3 -> GND
- J2 pad 23: GND -> /A8
- J2 pad 24: /D0 -> /RESET
- J2 pad 25: /D1 -> /A9
- J2 pad 26: /D2 -> /~{MREQ}
- J2 pad 27: /D3 -> /A10
- J2 pad 28: /D4 -> /~{IORQ}
- J2 pad 29: /D5 -> /A11
- J2 pad 3: /A2 -> GND
- J2 pad 30: /D6 -> /~{CBLK}
- J2 pad 31: /D7 -> /A12
- J2 pad 32: GND -> /~{BREQ}
- J2 pad 33: +5V -> /A13
- J2 pad 34: +5V -> /~{HALT}
- J2 pad 35: GND -> /A14
- J2 pad 36: /E -> /~{MRDY}
- J2 pad 37: /Q -> /A15
- J2 pad 38: /~{VMA} -> /~{ROM_{cs}}
- J2 pad 39: GND -> /~{MMU_{en}}
- J2 pad 4: /A3 -> GND
- J2 pad 40: /R/~{W} -> /~{RAM_{oe}}
- J2 pad 41: /~{RD} -> GND
- J2 pad 42: /~{WR} -> GND
- J2 pad 43: /~{RAM_{oe}} -> +3V3
- J2 pad 44: GND -> +3V3
- J2 pad 45: /~{CBLK} -> GND
- J2 pad 46: /~{IORQ} -> GND
- J2 pad 47: /~{MREQ} -> +12V
- J2 pad 48: /~{HALT} -> /BA
- J2 pad 49: /~{MRDY} -> -12V
- J2 pad 5: /A4 -> /A0
- J2 pad 50: /~{BREQ} -> /BS
- J2 pad 52: /BA -> GND
- J2 pad 53: /BS -> /D0
- J2 pad 54: /SPARE -> /USR1
- J2 pad 55: /~{RESET} -> /D1
- J2 pad 56: /~{NMI} -> /USR2
- J2 pad 57: /~{IRQ} -> /D2
- J2 pad 58: /~{FIRQ} -> /USR3
- J2 pad 59: GND -> /D3
- J2 pad 6: /A5 -> /Q
- J2 pad 60: +5V -> /USR4
- J2 pad 61: +5V -> /D4
- J2 pad 62: GND -> /~{RESET}
- J2 pad 7: /A6 -> /A1
- J2 pad 8: /A7 -> /E
- J2 pad 9: /A8 -> /A2
- J3 pad 1: /A0 -> +5V
- J3 pad 10: /A9 -> /~{RD}
- J3 pad 11: /A10 -> /A3
- J3 pad 12: /A11 -> /~{WR}
- J3 pad 13: /A12 -> /A4
- J3 pad 14: /A13 -> /R/~{W}
- J3 pad 15: /A14 -> /A5
- J3 pad 16: /A15 -> /~{CART_{en}}
- J3 pad 17: GND -> /A6
- J3 pad 18: -12V -> /CLK1
- J3 pad 19: +12V -> /A7
- J3 pad 2: /A1 -> +5V
- J3 pad 20: GND -> /CLK2
- J3 pad 21: +3V3 -> GND
- J3 pad 22: +3V3 -> GND
- J3 pad 23: GND -> /A8
- J3 pad 24: /D0 -> /RESET
- J3 pad 25: /D1 -> /A9
- J3 pad 26: /D2 -> /~{MREQ}
- J3 pad 27: /D3 -> /A10
- J3 pad 28: /D4 -> /~{IORQ}
- J3 pad 29: /D5 -> /A11
- J3 pad 3: /A2 -> GND
- J3 pad 30: /D6 -> /~{CBLK}
- J3 pad 31: /D7 -> /A12
- J3 pad 32: GND -> /~{BREQ}
- J3 pad 33: +5V -> /A13
- J3 pad 34: +5V -> /~{HALT}
- J3 pad 35: GND -> /A14
- J3 pad 36: /E -> /~{MRDY}
- J3 pad 37: /Q -> /A15
- J3 pad 38: /~{VMA} -> /~{ROM_{cs}}
- J3 pad 39: GND -> /~{MMU_{en}}
- J3 pad 4: /A3 -> GND
- J3 pad 40: /R/~{W} -> /~{RAM_{oe}}
- J3 pad 41: /~{RD} -> GND
- J3 pad 42: /~{WR} -> GND
- J3 pad 43: /~{RAM_{oe}} -> +3V3
- J3 pad 44: GND -> +3V3
- J3 pad 45: /~{CBLK} -> GND
- J3 pad 46: /~{IORQ} -> GND
- J3 pad 47: /~{MREQ} -> +12V
- J3 pad 48: /~{HALT} -> /BA
- J3 pad 49: /~{MRDY} -> -12V
- J3 pad 5: /A4 -> /A0
- J3 pad 50: /~{BREQ} -> /BS
- J3 pad 52: /BA -> GND
- J3 pad 53: /BS -> /D0
- J3 pad 54: /SPARE -> /USR1
- J3 pad 55: /~{RESET} -> /D1
- J3 pad 56: /~{NMI} -> /USR2
- J3 pad 57: /~{IRQ} -> /D2
- J3 pad 58: /~{FIRQ} -> /USR3
- J3 pad 59: GND -> /D3
- J3 pad 6: /A5 -> /Q
- J3 pad 60: +5V -> /USR4
- J3 pad 61: +5V -> /D4
- J3 pad 62: GND -> /~{RESET}
- J3 pad 7: /A6 -> /A1
- J3 pad 8: /A7 -> /E
- J3 pad 9: /A8 -> /A2
- J4 pad 1: /A0 -> +5V
- J4 pad 10: /A9 -> /~{RD}
- J4 pad 11: /A10 -> /A3
- J4 pad 12: /A11 -> /~{WR}
- J4 pad 13: /A12 -> /A4
- J4 pad 14: /A13 -> /R/~{W}
- J4 pad 15: /A14 -> /A5
- J4 pad 16: /A15 -> /~{CART_{en}}
- J4 pad 17: GND -> /A6
- J4 pad 18: -12V -> /CLK1
- J4 pad 19: +12V -> /A7
- J4 pad 2: /A1 -> +5V
- J4 pad 20: GND -> /CLK2
- J4 pad 21: +3V3 -> GND
- J4 pad 22: +3V3 -> GND
- J4 pad 23: GND -> /A8
- J4 pad 24: /D0 -> /RESET
- J4 pad 25: /D1 -> /A9
- J4 pad 26: /D2 -> /~{MREQ}
- J4 pad 27: /D3 -> /A10
- J4 pad 28: /D4 -> /~{IORQ}
- J4 pad 29: /D5 -> /A11
- J4 pad 3: /A2 -> GND
- J4 pad 30: /D6 -> /~{CBLK}
- J4 pad 31: /D7 -> /A12
- J4 pad 32: GND -> /~{BREQ}
- J4 pad 33: +5V -> /A13
- J4 pad 34: +5V -> /~{HALT}
- J4 pad 35: GND -> /A14
- J4 pad 36: /E -> /~{MRDY}
- J4 pad 37: /Q -> /A15
- J4 pad 38: /~{VMA} -> /~{ROM_{cs}}
- J4 pad 39: GND -> /~{MMU_{en}}
- J4 pad 4: /A3 -> GND
- J4 pad 40: /R/~{W} -> /~{RAM_{oe}}
- J4 pad 41: /~{RD} -> GND
- J4 pad 42: /~{WR} -> GND
- J4 pad 43: /~{RAM_{oe}} -> +3V3
- J4 pad 44: GND -> +3V3
- J4 pad 45: /~{CBLK} -> GND
- J4 pad 46: /~{IORQ} -> GND
- J4 pad 47: /~{MREQ} -> +12V
- J4 pad 48: /~{HALT} -> /BA
- J4 pad 49: /~{MRDY} -> -12V
- J4 pad 5: /A4 -> /A0
- J4 pad 50: /~{BREQ} -> /BS
- J4 pad 52: /BA -> GND
- J4 pad 53: /BS -> /D0
- J4 pad 54: /SPARE -> /USR1
- J4 pad 55: /~{RESET} -> /D1
- J4 pad 56: /~{NMI} -> /USR2
- J4 pad 57: /~{IRQ} -> /D2
- J4 pad 58: /~{FIRQ} -> /USR3
- J4 pad 59: GND -> /D3
- J4 pad 6: /A5 -> /Q
- J4 pad 60: +5V -> /USR4
- J4 pad 61: +5V -> /D4
- J4 pad 62: GND -> /~{RESET}
- J4 pad 7: /A6 -> /A1
- J4 pad 8: /A7 -> /E
- J4 pad 9: /A8 -> /A2
- J5 pad 1: /A0 -> +5V
- J5 pad 10: /A9 -> /~{RD}
- J5 pad 11: /A10 -> /A3
- J5 pad 12: /A11 -> /~{WR}
- J5 pad 13: /A12 -> /A4
- J5 pad 14: /A13 -> /R/~{W}
- J5 pad 15: /A14 -> /A5
- J5 pad 16: /A15 -> /~{CART_{en}}
- J5 pad 17: GND -> /A6
- J5 pad 18: -12V -> /CLK1
- J5 pad 19: +12V -> /A7
- J5 pad 2: /A1 -> +5V
- J5 pad 20: GND -> /CLK2
- J5 pad 21: +3V3 -> GND
- J5 pad 22: +3V3 -> GND
- J5 pad 23: GND -> /A8
- J5 pad 24: /D0 -> /RESET
- J5 pad 25: /D1 -> /A9
- J5 pad 26: /D2 -> /~{MREQ}
- J5 pad 27: /D3 -> /A10
- J5 pad 28: /D4 -> /~{IORQ}
- J5 pad 29: /D5 -> /A11
- J5 pad 3: /A2 -> GND
- J5 pad 30: /D6 -> /~{CBLK}
- J5 pad 31: /D7 -> /A12
- J5 pad 32: GND -> /~{BREQ}
- J5 pad 33: +5V -> /A13
- J5 pad 34: +5V -> /~{HALT}
- J5 pad 35: GND -> /A14
- J5 pad 36: /E -> /~{MRDY}
- J5 pad 37: /Q -> /A15
- J5 pad 38: /~{VMA} -> /~{ROM_{cs}}
- J5 pad 39: GND -> /~{MMU_{en}}
- J5 pad 4: /A3 -> GND
- J5 pad 40: /R/~{W} -> /~{RAM_{oe}}
- J5 pad 41: /~{RD} -> GND
- J5 pad 42: /~{WR} -> GND
- J5 pad 43: /~{RAM_{oe}} -> +3V3
- J5 pad 44: GND -> +3V3
- J5 pad 45: /~{CBLK} -> GND
- J5 pad 46: /~{IORQ} -> GND
- J5 pad 47: /~{MREQ} -> +12V
- J5 pad 48: /~{HALT} -> /BA
- J5 pad 49: /~{MRDY} -> -12V
- J5 pad 5: /A4 -> /A0
- J5 pad 50: /~{BREQ} -> /BS
- J5 pad 52: /BA -> GND
- J5 pad 53: /BS -> /D0
- J5 pad 54: /SPARE -> /USR1
- J5 pad 55: /~{RESET} -> /D1
- J5 pad 56: /~{NMI} -> /USR2
- J5 pad 57: /~{IRQ} -> /D2
- J5 pad 58: /~{FIRQ} -> /USR3
- J5 pad 59: GND -> /D3
- J5 pad 6: /A5 -> /Q
- J5 pad 60: +5V -> /USR4
- J5 pad 61: +5V -> /D4
- J5 pad 62: GND -> /~{RESET}
- J5 pad 7: /A6 -> /A1
- J5 pad 8: /A7 -> /E
- J5 pad 9: /A8 -> /A2
- J6 pad 1: /A0 -> +5V
- J6 pad 10: /A9 -> /~{RD}
- J6 pad 11: /A10 -> /A3
- J6 pad 12: /A11 -> /~{WR}
- J6 pad 13: /A12 -> /A4
- J6 pad 14: /A13 -> /R/~{W}
- J6 pad 15: /A14 -> /A5
- J6 pad 16: /A15 -> /~{CART_{en}}
- J6 pad 17: GND -> /A6
- J6 pad 18: -12V -> /CLK1
- J6 pad 19: +12V -> /A7
- J6 pad 2: /A1 -> +5V
- J6 pad 20: GND -> /CLK2
- J6 pad 21: +3V3 -> GND
- J6 pad 22: +3V3 -> GND
- J6 pad 23: GND -> /A8
- J6 pad 24: /D0 -> /RESET
- J6 pad 25: /D1 -> /A9
- J6 pad 26: /D2 -> /~{MREQ}
- J6 pad 27: /D3 -> /A10
- J6 pad 28: /D4 -> /~{IORQ}
- J6 pad 29: /D5 -> /A11
- J6 pad 3: /A2 -> GND
- J6 pad 30: /D6 -> /~{CBLK}
- J6 pad 31: /D7 -> /A12
- J6 pad 32: GND -> /~{BREQ}
- J6 pad 33: +5V -> /A13
- J6 pad 34: +5V -> /~{HALT}
- J6 pad 35: GND -> /A14
- J6 pad 36: /E -> /~{MRDY}
- J6 pad 37: /Q -> /A15
- J6 pad 38: /~{VMA} -> /~{ROM_{cs}}
- J6 pad 39: GND -> /~{MMU_{en}}
- J6 pad 4: /A3 -> GND
- J6 pad 40: /R/~{W} -> /~{RAM_{oe}}
- J6 pad 41: /~{RD} -> GND
- J6 pad 42: /~{WR} -> GND
- J6 pad 43: /~{RAM_{oe}} -> +3V3
- J6 pad 44: GND -> +3V3
- J6 pad 45: /~{CBLK} -> GND
- J6 pad 46: /~{IORQ} -> GND
- J6 pad 47: /~{MREQ} -> +12V
- J6 pad 48: /~{HALT} -> /BA
- J6 pad 49: /~{MRDY} -> -12V
- J6 pad 5: /A4 -> /A0
- J6 pad 50: /~{BREQ} -> /BS
- J6 pad 52: /BA -> GND
- J6 pad 53: /BS -> /D0
- J6 pad 54: /SPARE -> /USR1
- J6 pad 55: /~{RESET} -> /D1
- J6 pad 56: /~{NMI} -> /USR2
- J6 pad 57: /~{IRQ} -> /D2
- J6 pad 58: /~{FIRQ} -> /USR3
- J6 pad 59: GND -> /D3
- J6 pad 6: /A5 -> /Q
- J6 pad 60: +5V -> /USR4
- J6 pad 61: +5V -> /D4
- J6 pad 62: GND -> /~{RESET}
- J6 pad 7: /A6 -> /A1
- J6 pad 8: /A7 -> /E
- J6 pad 9: /A8 -> /A2
- J7 pad 1: /A0 -> +5V
- J7 pad 10: /E -> /~{RD}
- J7 pad 11: /A5 -> /A3
- J7 pad 12: /Q -> /~{WR}
- J7 pad 13: /A6 -> /A4
- J7 pad 14: /~{VMA} -> /R/~{W}
- J7 pad 15: /A7 -> /A5
- J7 pad 16: GND -> /~{CART_{en}}
- J7 pad 17: /A8 -> /A6
- J7 pad 18: /R/~{W} -> /CLK1
- J7 pad 19: /A9 -> /A7
- J7 pad 2: GND -> +5V
- J7 pad 20: /~{RD} -> /CLK2
- J7 pad 21: /A10 -> GND
- J7 pad 22: /~{WR} -> GND
- J7 pad 23: /A11 -> /A8
- J7 pad 24: /~{RAM_{oe}} -> /RESET
- J7 pad 25: /A12 -> /A9
- J7 pad 26: GND -> /~{MREQ}
- J7 pad 27: /A13 -> /A10
- J7 pad 28: /~{CBLK} -> /~{IORQ}
- J7 pad 29: /A14 -> /A11
- J7 pad 3: /A1 -> GND
- J7 pad 30: /~{IORQ} -> /~{CBLK}
- J7 pad 31: /A15 -> /A12
- J7 pad 32: /~{MREQ} -> /~{BREQ}
- J7 pad 33: GND -> /A13
- J7 pad 35: -12V -> /A14
- J7 pad 37: +12V -> /A15
- J7 pad 38: /~{BREQ} -> /~{ROM_{cs}}
- J7 pad 39: GND -> /~{MMU_{en}}
- J7 pad 4: +5V -> GND
- J7 pad 40: GND -> /~{RAM_{oe}}
- J7 pad 41: +3V3 -> GND
- J7 pad 42: /BA -> GND
- J7 pad 44: /BS -> +3V3
- J7 pad 46: /SPARE -> GND
- J7 pad 47: /D0 -> +12V
- J7 pad 48: /~{RESET} -> /BA
- J7 pad 49: /D1 -> -12V
- J7 pad 5: /A2 -> /A0
- J7 pad 50: /~{NMI} -> /BS
- J7 pad 51: /D2 -> GND
- J7 pad 52: /~{IRQ} -> GND
- J7 pad 53: /D3 -> /D0
- J7 pad 54: /~{FIRQ} -> /USR1
- J7 pad 55: /D4 -> /D1
- J7 pad 56: GND -> /USR2
- J7 pad 57: /D5 -> /D2
- J7 pad 58: +5V -> /USR3
- J7 pad 59: /D6 -> /D3
- J7 pad 6: +5V -> /Q
- J7 pad 60: +5V -> /USR4
- J7 pad 61: /D7 -> /D4
- J7 pad 62: GND -> /~{RESET}
- J7 pad 7: /A3 -> /A1
- J7 pad 8: GND -> /E
- J7 pad 9: /A4 -> /A2
- J9 pad 1: /A0 -> +5V
- J9 pad 10: /A9 -> /~{RD}
- J9 pad 11: /A10 -> /A3
- J9 pad 12: /A11 -> /~{WR}
- J9 pad 13: /A12 -> /A4
- J9 pad 14: /A13 -> /R/~{W}
- J9 pad 15: /A14 -> /A5
- J9 pad 16: /A15 -> /~{CART_{en}}
- J9 pad 17: GND -> /A6
- J9 pad 18: -12V -> /CLK1
- J9 pad 19: +12V -> /A7
- J9 pad 2: /A1 -> +5V
- J9 pad 20: GND -> /CLK2
- J9 pad 21: +3V3 -> GND
- J9 pad 22: +3V3 -> GND
- J9 pad 23: GND -> /A8
- J9 pad 24: /D0 -> /RESET
- J9 pad 25: /D1 -> /A9
- J9 pad 26: /D2 -> /~{MREQ}
- J9 pad 27: /D3 -> /A10
- J9 pad 28: /D4 -> /~{IORQ}
- J9 pad 29: /D5 -> /A11
- J9 pad 3: /A2 -> GND
- J9 pad 30: /D6 -> /~{CBLK}
- J9 pad 31: /D7 -> /A12
- J9 pad 32: GND -> /~{BREQ}
- J9 pad 33: +5V -> /A13
- J9 pad 34: +5V -> /~{HALT}
- J9 pad 35: GND -> /A14
- J9 pad 36: /E -> /~{MRDY}
- J9 pad 37: /Q -> /A15
- J9 pad 38: /~{VMA} -> /~{ROM_{cs}}
- J9 pad 39: GND -> /~{MMU_{en}}
- J9 pad 4: /A3 -> GND
- J9 pad 40: /R/~{W} -> /~{RAM_{oe}}
- J9 pad 41: /~{RD} -> GND
- J9 pad 42: /~{WR} -> GND
- J9 pad 43: /~{RAM_{oe}} -> +3V3
- J9 pad 44: GND -> +3V3
- J9 pad 45: /~{CBLK} -> GND
- J9 pad 46: /~{IORQ} -> GND
- J9 pad 47: /~{MREQ} -> +12V
- J9 pad 48: /~{HALT} -> /BA
- J9 pad 49: /~{MRDY} -> -12V
- J9 pad 5: /A4 -> /A0
- J9 pad 50: /~{BREQ} -> /BS
- J9 pad 52: /BA -> GND
- J9 pad 53: /BS -> /D0
- J9 pad 54: /SPARE -> /USR1
- J9 pad 55: /~{RESET} -> /D1
- J9 pad 56: /~{NMI} -> /USR2
- J9 pad 57: /~{IRQ} -> /D2
- J9 pad 58: /~{FIRQ} -> /USR3
- J9 pad 59: GND -> /D3
- J9 pad 6: /A5 -> /Q
- J9 pad 60: +5V -> /USR4
- J9 pad 61: +5V -> /D4
- J9 pad 62: GND -> /~{RESET}
- J9 pad 7: /A6 -> /A1
- J9 pad 8: /A7 -> /E
- J9 pad 9: /A8 -> /A2
- R3 pad 1: Net-(R2-Pad2) -> Net-(SW1-A)
- R3 pad 2: Net-(C2-Pad1) -> +5V
- R4 pad 1: Net-(SW1-A) -> Net-(R2-Pad2)
- R4 pad 2: +5V -> Net-(C2-Pad1)
- SW1 pad 3: GND -> Net-(R2-Pad2)
- SW1 pad 4: Net-(SW1-A) -> GND
- U2 pad 5: /Power/~{PS_ON} -> /~{PS_ON}
Other:
- board size 282.6 x 114.3 mm -> 285.8 x 124.5 mm
- board text added: "+5V"

Commit message: Placed bus traces
Parts:
- moved H3 327.4 mm to (53.3, 143.5)
- moved H1 326.6 mm to (53.3, 31.8)
- moved C177 292.6 mm to (30.5, 142.2), turned to -90 degrees
- moved H7 276.3 mm to (114.3, 31.8)
- moved H10 239.1 mm to (153.0, 166.4)
- moved H5 239.1 mm to (144.4, 166.4)
- moved H9 239.1 mm to (153.0, 157.9)
- moved H4 239.1 mm to (144.4, 157.9)
- moved H6 214.8 mm to (175.3, 31.8)
- moved C10 154.7 mm to (42.5, 33.0), turned to 90 degrees
- moved H2 150.3 mm to (236.2, 31.8)
- moved C187 114.4 mm to (42.5, 142.2), turned to -90 degrees
- moved H8 107.6 mm to (297.2, 31.8)
- moved SW1 91.6 mm to (333.4, 141.0)
- moved J8 88.7 mm to (306.2, 64.4), turned to 90 degrees
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Routing:
- net GND: track 0.00 -> 1469.3 mm
- net +5V: track 0.00 -> 489.8 mm
- net /A11: track 0.00 -> 255.2 mm
- net /D7: track 0.00 -> 255.2 mm
- net /D6: track 0.00 -> 255.2 mm
- net /D4: track 0.00 -> 255.2 mm
- net /A9: track 0.00 -> 255.2 mm
- net +12V: track 0.00 -> 255.2 mm
- net /A1: track 0.00 -> 255.2 mm
- net /A0: track 0.00 -> 255.2 mm
- net /A13: track 0.00 -> 255.2 mm
- net /D2: track 0.00 -> 255.2 mm
- net /D3: track 0.00 -> 255.2 mm
- net /A7: track 0.00 -> 255.2 mm
- net /D0: track 0.00 -> 255.2 mm
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