File: Episode4/Episode4.kicad_pcb (KiCad board)
At the start: 2 copper layers, 285.8 x 124.5 mm, 231 parts, among them J1 CARD, J10 CARD, J11 CARD, J12 CARD, J13 CARD, J14 CARD, J2 CARD, J3 CARD, J4 CARD, J5 CARD, J6 CARD, J7 BB Con, J8 ATX POWER, J9 CARD, SW1 POWER, U1 74HCT14, U2 74HCT74

Commit message: Added various IRQ and FIRQ lines
Connections:
- net /USR3 renamed /~{IRQ2}
- net /USR4 renamed /~{IRQ3}
- net /~{IRQ} renamed /~{IRQ7}
- J1 pad 10: /~{RD} -> /~{RESET}
- J1 pad 12: /~{WR} -> /~{RD}
- J1 pad 14: /R/~{W} -> /~{WR}
- J1 pad 16: /~{CART_{en}} -> /R/~{W}
- J1 pad 18: /CLK1 -> /USR1
- J1 pad 20: /CLK2 -> /USR2
- J1 pad 24: /RESET -> /~{MREQ}
- J1 pad 26: /~{MREQ} -> /~{IORQ}
- J1 pad 28: /~{IORQ} -> /~{CBLK}
- J1 pad 30: /~{CBLK} -> /~{BREQ}
- J1 pad 32: /~{BREQ} -> /~{HALT}
- J1 pad 34: /~{HALT} -> /~{MRDY}
- J1 pad 36: /~{MRDY} -> /BA
- J1 pad 38: /~{ROM_{cs}} -> /BS
- J1 pad 48: /BA -> /FIRQ1
- J1 pad 50: /BS -> /FIRQ2
- J1 pad 54: /USR1 -> /FIRQ3
- J1 pad 56: /USR2 -> /~{IRQ1}
- J1 pad 62: /~{RESET} -> /~{IRQ5}
- J1 pad 64: /~{NMI} -> /~{IRQ6}
- J1 pad 68: /~{FIRQ} -> /~{NMI}
- J10 pad 10: /~{RD} -> /~{RESET}
- J10 pad 12: /~{WR} -> /~{RD}
- J10 pad 14: /R/~{W} -> /~{WR}
- J10 pad 16: /~{CART_{en}} -> /R/~{W}
- J10 pad 18: /CLK1 -> /USR1
- J10 pad 20: /CLK2 -> /USR2
- J10 pad 24: /RESET -> /~{MREQ}
- J10 pad 26: /~{MREQ} -> /~{IORQ}
- J10 pad 28: /~{IORQ} -> /~{CBLK}
- J10 pad 30: /~{CBLK} -> /~{BREQ}
- J10 pad 32: /~{BREQ} -> /~{HALT}
- J10 pad 34: /~{HALT} -> /~{MRDY}
- J10 pad 36: /~{MRDY} -> /BA
- J10 pad 38: /~{ROM_{cs}} -> /BS
- J10 pad 48: /BA -> /FIRQ1
- J10 pad 50: /BS -> /FIRQ2
- J10 pad 54: /USR1 -> /FIRQ3
- J10 pad 56: /USR2 -> /~{IRQ1}
- J10 pad 62: /~{RESET} -> /~{IRQ5}
- J10 pad 64: /~{NMI} -> /~{IRQ6}
- J10 pad 68: /~{FIRQ} -> /~{NMI}
- J11 pad 10: /~{RD} -> /~{RESET}
- J11 pad 12: /~{WR} -> /~{RD}
- J11 pad 14: /R/~{W} -> /~{WR}
- J11 pad 16: /~{CART_{en}} -> /R/~{W}
- J11 pad 18: /CLK1 -> /USR1
- J11 pad 20: /CLK2 -> /USR2
- J11 pad 24: /RESET -> /~{MREQ}
- J11 pad 26: /~{MREQ} -> /~{IORQ}
- J11 pad 28: /~{IORQ} -> /~{CBLK}
- J11 pad 30: /~{CBLK} -> /~{BREQ}
- J11 pad 32: /~{BREQ} -> /~{HALT}
- J11 pad 34: /~{HALT} -> /~{MRDY}
- J11 pad 36: /~{MRDY} -> /BA
- J11 pad 38: /~{ROM_{cs}} -> /BS
- J11 pad 48: /BA -> /FIRQ1
- J11 pad 50: /BS -> /FIRQ2
- J11 pad 54: /USR1 -> /FIRQ3
- J11 pad 56: /USR2 -> /~{IRQ1}
- J11 pad 62: /~{RESET} -> /~{IRQ5}
- J11 pad 64: /~{NMI} -> /~{IRQ6}
- J11 pad 68: /~{FIRQ} -> /~{NMI}
- J12 pad 10: /~{RD} -> /~{RESET}
- J12 pad 12: /~{WR} -> /~{RD}
- J12 pad 14: /R/~{W} -> /~{WR}
- J12 pad 16: /~{CART_{en}} -> /R/~{W}
- J12 pad 18: /CLK1 -> /USR1
- J12 pad 20: /CLK2 -> /USR2
- J12 pad 24: /RESET -> /~{MREQ}
- J12 pad 26: /~{MREQ} -> /~{IORQ}
- J12 pad 28: /~{IORQ} -> /~{CBLK}
- J12 pad 30: /~{CBLK} -> /~{BREQ}
- J12 pad 32: /~{BREQ} -> /~{HALT}
- J12 pad 34: /~{HALT} -> /~{MRDY}
- J12 pad 36: /~{MRDY} -> /BA
- J12 pad 38: /~{ROM_{cs}} -> /BS
- J12 pad 48: /BA -> /FIRQ1
- J12 pad 50: /BS -> /FIRQ2
- J12 pad 54: /USR1 -> /FIRQ3
- J12 pad 56: /USR2 -> /~{IRQ1}
- J12 pad 62: /~{RESET} -> /~{IRQ5}
- J12 pad 64: /~{NMI} -> /~{IRQ6}
- J12 pad 68: /~{FIRQ} -> /~{NMI}
- J13 pad 10: /~{RD} -> /~{RESET}
- J13 pad 12: /~{WR} -> /~{RD}
- J13 pad 14: /R/~{W} -> /~{WR}
- J13 pad 16: /~{CART_{en}} -> /R/~{W}
- J13 pad 18: /CLK1 -> /USR1
- J13 pad 20: /CLK2 -> /USR2
- J13 pad 24: /RESET -> /~{MREQ}
- J13 pad 26: /~{MREQ} -> /~{IORQ}
- J13 pad 28: /~{IORQ} -> /~{CBLK}
- J13 pad 30: /~{CBLK} -> /~{BREQ}
- J13 pad 32: /~{BREQ} -> /~{HALT}
- J13 pad 34: /~{HALT} -> /~{MRDY}
- J13 pad 36: /~{MRDY} -> /BA
- J13 pad 38: /~{ROM_{cs}} -> /BS
- J13 pad 48: /BA -> /FIRQ1
- J13 pad 50: /BS -> /FIRQ2
- J13 pad 54: /USR1 -> /FIRQ3
- J13 pad 56: /USR2 -> /~{IRQ1}
- J13 pad 62: /~{RESET} -> /~{IRQ5}
- J13 pad 64: /~{NMI} -> /~{IRQ6}
- J13 pad 68: /~{FIRQ} -> /~{NMI}
- J14 pad 10: /~{RD} -> /~{RESET}
- J14 pad 12: /~{WR} -> /~{RD}
- J14 pad 14: /R/~{W} -> /~{WR}
- J14 pad 16: /~{CART_{en}} -> /R/~{W}
- J14 pad 18: /CLK1 -> /USR1
- J14 pad 20: /CLK2 -> /USR2
- J14 pad 24: /RESET -> /~{MREQ}
- J14 pad 26: /~{MREQ} -> /~{IORQ}
- J14 pad 28: /~{IORQ} -> /~{CBLK}
- J14 pad 30: /~{CBLK} -> /~{BREQ}
- J14 pad 32: /~{BREQ} -> /~{HALT}
- J14 pad 34: /~{HALT} -> /~{MRDY}
- J14 pad 36: /~{MRDY} -> /BA
- J14 pad 38: /~{ROM_{cs}} -> /BS
- J14 pad 48: /BA -> /FIRQ1
- J14 pad 50: /BS -> /FIRQ2
- J14 pad 54: /USR1 -> /FIRQ3
- J14 pad 56: /USR2 -> /~{IRQ1}
- J14 pad 62: /~{RESET} -> /~{IRQ5}
- J14 pad 64: /~{NMI} -> /~{IRQ6}
- J14 pad 68: /~{FIRQ} -> /~{NMI}
- J2 pad 10: /~{RD} -> /~{RESET}
- J2 pad 12: /~{WR} -> /~{RD}
- J2 pad 14: /R/~{W} -> /~{WR}
- J2 pad 16: /~{CART_{en}} -> /R/~{W}
- J2 pad 18: /CLK1 -> /USR1
- J2 pad 20: /CLK2 -> /USR2
- J2 pad 24: /RESET -> /~{MREQ}
- J2 pad 26: /~{MREQ} -> /~{IORQ}
- J2 pad 28: /~{IORQ} -> /~{CBLK}
- J2 pad 30: /~{CBLK} -> /~{BREQ}
- J2 pad 32: /~{BREQ} -> /~{HALT}
- J2 pad 34: /~{HALT} -> /~{MRDY}
- J2 pad 36: /~{MRDY} -> /BA
- J2 pad 38: /~{ROM_{cs}} -> /BS
- J2 pad 48: /BA -> /FIRQ1
- J2 pad 50: /BS -> /FIRQ2
- J2 pad 54: /USR1 -> /FIRQ3
- J2 pad 56: /USR2 -> /~{IRQ1}
- J2 pad 62: /~{RESET} -> /~{IRQ5}
- J2 pad 64: /~{NMI} -> /~{IRQ6}
- J2 pad 68: /~{FIRQ} -> /~{NMI}
- J3 pad 10: /~{RD} -> /~{RESET}
- J3 pad 12: /~{WR} -> /~{RD}
- J3 pad 14: /R/~{W} -> /~{WR}
- J3 pad 16: /~{CART_{en}} -> /R/~{W}
- J3 pad 18: /CLK1 -> /USR1
- J3 pad 20: /CLK2 -> /USR2
- J3 pad 24: /RESET -> /~{MREQ}
- J3 pad 26: /~{MREQ} -> /~{IORQ}
- J3 pad 28: /~{IORQ} -> /~{CBLK}
- J3 pad 30: /~{CBLK} -> /~{BREQ}
- J3 pad 32: /~{BREQ} -> /~{HALT}
- J3 pad 34: /~{HALT} -> /~{MRDY}
- J3 pad 36: /~{MRDY} -> /BA
- J3 pad 38: /~{ROM_{cs}} -> /BS
- J3 pad 48: /BA -> /FIRQ1
- J3 pad 50: /BS -> /FIRQ2
- J3 pad 54: /USR1 -> /FIRQ3
- J3 pad 56: /USR2 -> /~{IRQ1}
- J3 pad 62: /~{RESET} -> /~{IRQ5}
- J3 pad 64: /~{NMI} -> /~{IRQ6}
- J3 pad 68: /~{FIRQ} -> /~{NMI}
- J4 pad 10: /~{RD} -> /~{RESET}
- J4 pad 12: /~{WR} -> /~{RD}
- J4 pad 14: /R/~{W} -> /~{WR}
- J4 pad 16: /~{CART_{en}} -> /R/~{W}
- J4 pad 18: /CLK1 -> /USR1
- J4 pad 20: /CLK2 -> /USR2
- J4 pad 24: /RESET -> /~{MREQ}
- J4 pad 26: /~{MREQ} -> /~{IORQ}
- J4 pad 28: /~{IORQ} -> /~{CBLK}
- J4 pad 30: /~{CBLK} -> /~{BREQ}
- J4 pad 32: /~{BREQ} -> /~{HALT}
- J4 pad 34: /~{HALT} -> /~{MRDY}
- J4 pad 36: /~{MRDY} -> /BA
- J4 pad 38: /~{ROM_{cs}} -> /BS
- J4 pad 48: /BA -> /FIRQ1
- J4 pad 50: /BS -> /FIRQ2
- J4 pad 54: /USR1 -> /FIRQ3
- J4 pad 56: /USR2 -> /~{IRQ1}
- J4 pad 62: /~{RESET} -> /~{IRQ5}
- J4 pad 64: /~{NMI} -> /~{IRQ6}
- J4 pad 68: /~{FIRQ} -> /~{NMI}
- J5 pad 10: /~{RD} -> /~{RESET}
- J5 pad 12: /~{WR} -> /~{RD}
- J5 pad 14: /R/~{W} -> /~{WR}
- J5 pad 16: /~{CART_{en}} -> /R/~{W}
- J5 pad 18: /CLK1 -> /USR1
- J5 pad 20: /CLK2 -> /USR2
- J5 pad 24: /RESET -> /~{MREQ}
- J5 pad 26: /~{MREQ} -> /~{IORQ}
- J5 pad 28: /~{IORQ} -> /~{CBLK}
- J5 pad 30: /~{CBLK} -> /~{BREQ}
- J5 pad 32: /~{BREQ} -> /~{HALT}
- J5 pad 34: /~{HALT} -> /~{MRDY}
- J5 pad 36: /~{MRDY} -> /BA
- J5 pad 38: /~{ROM_{cs}} -> /BS
- J5 pad 48: /BA -> /FIRQ1
- J5 pad 50: /BS -> /FIRQ2
- J5 pad 54: /USR1 -> /FIRQ3
- J5 pad 56: /USR2 -> /~{IRQ1}
- J5 pad 62: /~{RESET} -> /~{IRQ5}
- J5 pad 64: /~{NMI} -> /~{IRQ6}
- J5 pad 68: /~{FIRQ} -> /~{NMI}
- J6 pad 10: /~{RD} -> /~{RESET}
- J6 pad 12: /~{WR} -> /~{RD}
- J6 pad 14: /R/~{W} -> /~{WR}
- J6 pad 16: /~{CART_{en}} -> /R/~{W}
- J6 pad 18: /CLK1 -> /USR1
- J6 pad 20: /CLK2 -> /USR2
- J6 pad 24: /RESET -> /~{MREQ}
- J6 pad 26: /~{MREQ} -> /~{IORQ}
- J6 pad 28: /~{IORQ} -> /~{CBLK}
- J6 pad 30: /~{CBLK} -> /~{BREQ}
- J6 pad 32: /~{BREQ} -> /~{HALT}
- J6 pad 34: /~{HALT} -> /~{MRDY}
- J6 pad 36: /~{MRDY} -> /BA
- J6 pad 38: /~{ROM_{cs}} -> /BS
- J6 pad 48: /BA -> /FIRQ1
- J6 pad 50: /BS -> /FIRQ2
- J6 pad 54: /USR1 -> /FIRQ3
- J6 pad 56: /USR2 -> /~{IRQ1}
- J6 pad 62: /~{RESET} -> /~{IRQ5}
- J6 pad 64: /~{NMI} -> /~{IRQ6}
- J6 pad 68: /~{FIRQ} -> /~{NMI}
- J7 pad 10: /~{RD} -> /~{RESET}
- J7 pad 12: /~{WR} -> /~{RD}
- J7 pad 14: /R/~{W} -> /~{WR}
- J7 pad 16: /~{CART_{en}} -> /R/~{W}
- J7 pad 18: /CLK1 -> /USR1
- J7 pad 20: /CLK2 -> /USR2
- J7 pad 24: /RESET -> /~{MREQ}
- J7 pad 26: /~{MREQ} -> /~{IORQ}
- J7 pad 28: /~{IORQ} -> /~{CBLK}
- J7 pad 30: /~{CBLK} -> /~{BREQ}
- J7 pad 32: /~{BREQ} -> /~{HALT}
- J7 pad 34: /~{HALT} -> /~{MRDY}
- J7 pad 36: /~{MRDY} -> /BA
- J7 pad 38: /~{ROM_{cs}} -> /BS
- J7 pad 48: /BA -> /FIRQ1
- J7 pad 50: /BS -> /FIRQ2
- J7 pad 54: /USR1 -> /FIRQ3
- J7 pad 56: /USR2 -> /~{IRQ1}
- J7 pad 62: /~{RESET} -> /~{IRQ5}
- J7 pad 64: /~{NMI} -> /~{IRQ6}
- J7 pad 68: /~{FIRQ} -> /~{NMI}
- J9 pad 10: /~{RD} -> /~{RESET}
- J9 pad 12: /~{WR} -> /~{RD}
- J9 pad 14: /R/~{W} -> /~{WR}
- J9 pad 16: /~{CART_{en}} -> /R/~{W}
- J9 pad 18: /CLK1 -> /USR1
- J9 pad 20: /CLK2 -> /USR2
- J9 pad 24: /RESET -> /~{MREQ}
- J9 pad 26: /~{MREQ} -> /~{IORQ}
- J9 pad 28: /~{IORQ} -> /~{CBLK}
- J9 pad 30: /~{CBLK} -> /~{BREQ}
- J9 pad 32: /~{BREQ} -> /~{HALT}
- J9 pad 34: /~{HALT} -> /~{MRDY}
- J9 pad 36: /~{MRDY} -> /BA
- J9 pad 38: /~{ROM_{cs}} -> /BS
- J9 pad 48: /BA -> /FIRQ1
- J9 pad 50: /BS -> /FIRQ2
- J9 pad 54: /USR1 -> /FIRQ3
- J9 pad 56: /USR2 -> /~{IRQ1}
- J9 pad 62: /~{RESET} -> /~{IRQ5}
- J9 pad 64: /~{NMI} -> /~{IRQ6}
- J9 pad 68: /~{FIRQ} -> /~{NMI}
Routing:
- net /~{ROM_{cs}}: track 252.7 -> 0.00 mm
- net /~{IRQ1}: track 0.00 -> 252.7 mm
- net /~{CART_{en}}: track 252.7 -> 0.00 mm
- net /RESET: track 252.7 -> 0.00 mm
- net /CLK2: track 252.7 -> 0.00 mm
- net /CLK1: track 252.7 -> 0.00 mm
- net /~{IRQ5}: track 0.00 -> 252.7 mm
- net /~{IRQ6}: track 0.00 -> 252.7 mm
- net /~{FIRQ}: track 252.7 -> 0.00 mm
- net /FIRQ3: track 0.00 -> 252.7 mm
- net /FIRQ2: track 0.00 -> 252.7 mm
- net /FIRQ1: track 0.00 -> 252.7 mm

Commit message: Shuffled around IRQ numbers, and removed NMI, as it will by on the CPU card only.
Parts:
- moved C1 162.0 mm to (247.8, 164.7)
- moved C2 162.0 mm to (247.8, 167.7)
- moved U1 162.0 mm to (244.8, 158.1)
- moved R1 162.0 mm to (243.0, 164.7)
- moved R2 162.0 mm to (243.0, 167.6)
- moved R3 162.0 mm to (243.0, 170.6)
- moved R4 162.0 mm to (243.0, 173.5)
- moved U2 162.0 mm to (253.3, 158.1)
- moved H10 126.0 mm to (276.9, 143.5)
- moved H5 75.0 mm to (215.9, 143.5)
- moved H4 52.5 mm to (94.0, 143.5)
- moved H9 14.5 mm to (154.9, 143.5)
Connections:
- J1 pad 62: /~{IRQ5} -> /~{IRQ4}
- J1 pad 64: /~{IRQ6} -> /~{IRQ5}
- J1 pad 66: /~{IRQ7} -> /~{IRQ6}
- J1 pad 68: /~{NMI} -> /~{IRQ7}
- J10 pad 62: /~{IRQ5} -> /~{IRQ4}
- J10 pad 64: /~{IRQ6} -> /~{IRQ5}
- J10 pad 66: /~{IRQ7} -> /~{IRQ6}
- J10 pad 68: /~{NMI} -> /~{IRQ7}
- J11 pad 62: /~{IRQ5} -> /~{IRQ4}
- J11 pad 64: /~{IRQ6} -> /~{IRQ5}
- J11 pad 66: /~{IRQ7} -> /~{IRQ6}
- J11 pad 68: /~{NMI} -> /~{IRQ7}
- J12 pad 62: /~{IRQ5} -> /~{IRQ4}
- J12 pad 64: /~{IRQ6} -> /~{IRQ5}
- J12 pad 66: /~{IRQ7} -> /~{IRQ6}
- J12 pad 68: /~{NMI} -> /~{IRQ7}
- J13 pad 62: /~{IRQ5} -> /~{IRQ4}
- J13 pad 64: /~{IRQ6} -> /~{IRQ5}
- J13 pad 66: /~{IRQ7} -> /~{IRQ6}
- J13 pad 68: /~{NMI} -> /~{IRQ7}
- J14 pad 62: /~{IRQ5} -> /~{IRQ4}
- J14 pad 64: /~{IRQ6} -> /~{IRQ5}
- J14 pad 66: /~{IRQ7} -> /~{IRQ6}
- J14 pad 68: /~{NMI} -> /~{IRQ7}
- J2 pad 62: /~{IRQ5} -> /~{IRQ4}
- J2 pad 64: /~{IRQ6} -> /~{IRQ5}
- J2 pad 66: /~{IRQ7} -> /~{IRQ6}
- J2 pad 68: /~{NMI} -> /~{IRQ7}
- J3 pad 62: /~{IRQ5} -> /~{IRQ4}
- J3 pad 64: /~{IRQ6} -> /~{IRQ5}
- J3 pad 66: /~{IRQ7} -> /~{IRQ6}
- J3 pad 68: /~{NMI} -> /~{IRQ7}
- J4 pad 62: /~{IRQ5} -> /~{IRQ4}
- J4 pad 64: /~{IRQ6} -> /~{IRQ5}
- J4 pad 66: /~{IRQ7} -> /~{IRQ6}
- J4 pad 68: /~{NMI} -> /~{IRQ7}
- J5 pad 62: /~{IRQ5} -> /~{IRQ4}
- J5 pad 64: /~{IRQ6} -> /~{IRQ5}
- J5 pad 66: /~{IRQ7} -> /~{IRQ6}
- J5 pad 68: /~{NMI} -> /~{IRQ7}
- J6 pad 62: /~{IRQ5} -> /~{IRQ4}
- J6 pad 64: /~{IRQ6} -> /~{IRQ5}
- J6 pad 66: /~{IRQ7} -> /~{IRQ6}
- J6 pad 68: /~{NMI} -> /~{IRQ7}
- J7 pad 62: /~{IRQ5} -> /~{IRQ4}
- J7 pad 64: /~{IRQ6} -> /~{IRQ5}
- J7 pad 66: /~{IRQ7} -> /~{IRQ6}
- J7 pad 68: /~{NMI} -> /~{IRQ7}
- J9 pad 62: /~{IRQ5} -> /~{IRQ4}
- J9 pad 64: /~{IRQ6} -> /~{IRQ5}
- J9 pad 66: /~{IRQ7} -> /~{IRQ6}
- J9 pad 68: /~{NMI} -> /~{IRQ7}
Routing:
- net /~{IRQ4}: track 0.00 -> 252.7 mm
- net /~{NMI}: track 252.7 -> 0.00 mm

Commit message: Changed data trace width, and moving power lanes to inner power plane.
Parts:
- D1, D2, D3, D4, D5, D6, D7, D8: moved to B.Cu
- moved D5 343.9 mm to (28.6, 43.2), turned to 180 degrees
- moved D6 339.7 mm to (28.6, 96.5), turned to 180 degrees
- moved D7 339.7 mm to (28.6, 102.9), turned to 180 degrees
- moved D8 339.7 mm to (28.6, 109.2)
- moved C32 268.7 mm to (266.7, 49.5), turned to -90 degrees
- moved C62 266.8 mm to (246.4, 110.5), turned to 90 degrees
- moved C58 266.7 mm to (266.7, 110.5), turned to -90 degrees
- moved C23 257.6 mm to (246.4, 49.5), turned to -90 degrees
- moved C46 247.0 mm to (266.7, 92.1), turned to 90 degrees
- moved C40 231.4 mm to (225.9, 49.5), turned to -90 degrees
- moved C61 231.0 mm to (205.7, 110.5), turned to 90 degrees
- moved C45 229.4 mm to (246.4, 92.1), turned to 90 degrees
- moved C57 228.4 mm to (226.1, 110.5), turned to -90 degrees
- moved C41 224.1 mm to (266.7, 125.7), turned to 90 degrees
- moved C31 221.5 mm to (205.6, 49.5), turned to -90 degrees
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Routing:
- net +5V: track 489.8 -> 0.00 mm
- net +12V: track 255.2 -> 236.8 mm
- net -12V: track 255.2 -> 236.8 mm
Other:
- copper layers 2 -> 4

Commit message: Reworked bus line order, capacitor and trace placement
Parts:
- removed the C13 at (330.8, 59.1)
- removed the C176 at (30.5, 33.0)
- removed the C177 at (30.5, 142.2)
- removed the C183 at (289.0, 84.5)
- removed the C186 at (13.3, 96.0)
- removed the C187 at (42.5, 142.2)
- removed the C190 at (63.5, 142.2)
- removed the D1 at (325.1, 132.7)
- removed the D2 at (325.1, 96.5)
- removed the D3 at (325.1, 102.9)
- removed the D4 at (325.1, 109.2)
- added C10: .01µF, Capacitor_SMD:C_0805_2012Metric_Pad1.18x1.45mm_HandSolder, F.Cu at (374.1, 76.9)
- added C11: .01µF, Capacitor_SMD:C_0805_2012Metric_Pad1.18x1.45mm_HandSolder, F.Cu at (374.1, 79.9)
- added C15: .01µF, Capacitor_SMD:C_0805_2012Metric_Pad1.18x1.45mm_HandSolder, F.Cu at (374.1, 82.9)
- added C19: .01µF, Capacitor_SMD:C_0805_2012Metric_Pad1.18x1.45mm_HandSolder, F.Cu at (374.1, 89.0)
- added C23: .01µF, Capacitor_SMD:C_0805_2012Metric_Pad1.18x1.45mm_HandSolder, F.Cu at (374.1, 85.9)
- added C46: 10µF, Capacitor_SMD:CP_Elec_4x5.8, F.Cu at (43.2, 44.5)
- added C47: 10µF, Capacitor_SMD:CP_Elec_4x5.8, F.Cu at (43.2, 130.8)
- added C59: 10µF, Capacitor_SMD:CP_Elec_4x5.8, F.Cu at (43.2, 95.2)
- added C71: 10µF, Capacitor_SMD:CP_Elec_4x5.8, F.Cu at (43.2, 103.5)
- added D5: TVS 5V, Diode_SMD:D_SMB, B.Cu at (3.72, 119.4)
- C12: renamed from C10; value 100µF -> 220µF
- C3, C4: value 100µF -> 220µF
- moved C12 249.8 mm to (289.6, 70.5)
- moved H1 30.5 mm to (22.9, 31.8)
- moved H3 30.5 mm to (22.9, 143.5)
- moved D3 25.2 mm to (3.42, 101.0)
- moved U1 24.8 mm to (261.0, 142.9)
- moved C182 24.8 mm to (254.0, 142.9)
- moved C183 24.8 mm to (274.3, 142.9)
- moved U2 24.8 mm to (281.3, 142.9)
- moved D4 24.5 mm to (4.05, 109.2)
- moved SW1 22.2 mm to (308.4, 118.1)
- moved D2 22.0 mm to (6.59, 95.9)
- moved H4 20.3 mm to (94.0, 143.5)
- moved H7 20.3 mm to (94.0, 31.8)
- moved C4 19.1 mm to (289.6, 130.8)
- moved D1 18.2 mm to (10.4, 43.2)
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- renumbered C92 to C100, C93 to C101, C94 to C102, C95 to C103, C96 to C104, C97 to C105, C98 to C106, C99 to C107, C100 to C108, C101 to C109, C102 to C110, C103 to C111, C104 to C112, C105 to C113, C106 to C114, C107 to C115, C108 to C116, C109 to C117, C110 to C118, C111 to C119, C112 to C120, C113 to C121, C114 to C122, C115 to C123, C116 to C124, C117 to C125, C118 to C126, C119 to C127, C120 to C128, C121 to C129, C11 to C13, C122 to C130, C123 to C131, C124 to C132, C125 to C133, C126 to C134, C127 to C135, C128 to C136, C129 to C137, C130 to C138, C131 to C139, C12 to C14, C132 to C140, C133 to C141, C134 to C142, C135 to C143, C136 to C144, C137 to C145, C138 to C146, C139 to C147, C140 to C148, C141 to C149, C142 to C150, C143 to C151, C144 to C152, C145 to C153, C146 to C154, C147 to C155, C148 to C156, C149 to C157, C150 to C158, C151 to C159, C14 to C16, C152 to C160, C153 to C161, C154 to C162, C155 to C163, C156 to C164, C157 to C165, C158 to C166, C159 to C167, C160 to C168, C161 to C169, C15 to C17, C162 to C170, C163 to C171, C164 to C172, C165 to C173, C166 to C174, C167 to C175, C168 to C176, C169 to C177, C170 to C178, C171 to C179, C16 to C18, C172 to C180, C173 to C181, C174 to C182, C175 to C183, C178 to C184, C179 to C185, C180 to C186, C181 to C187, C182 to C188, C184 to C189, C185 to C190, C188 to C191, C189 to C192, C191 to C193, C192 to C194, C17 to C20, C18 to C21, C19 to C22, C20 to C24, C21 to C25, C22 to C26, C23 to C27, C24 to C28, C25 to C29, C26 to C30, C27 to C31, C28 to C32, C29 to C33, C30 to C34, C31 to C35, C32 to C36, C33 to C37, C34 to C38, C35 to C39, C36 to C40, C37 to C41, C38 to C42, C39 to C43, C40 to C44, C41 to C45, C42 to C48, C43 to C49, C44 to C50, C45 to C51, C46 to C52, C47 to C53, C48 to C54, C49 to C55, C50 to C56, C51 to C57, C52 to C58, C53 to C60, C54 to C61, C55 to C62, C56 to C63, C57 to C64, C58 to C65, C59 to C66, C60 to C67, C61 to C68, C62 to C69, C63 to C70, C64 to C72, C65 to C73, C66 to C74, C67 to C75, C68 to C76, C69 to C77, C70 to C78, C71 to C79, C72 to C80, C73 to C81, C74 to C82, C75 to C83, C76 to C84, C77 to C85, C78 to C86, C79 to C87, C80 to C88, C81 to C89, C82 to C90, C83 to C91, C84 to C92, C85 to C93, C86 to C94, C87 to C95, C88 to C96, C89 to C97, C90 to C98, C91 to C99, D5 to D1, D6 to D2, D7 to D3, D8 to D4, J8 to J7, J7 to J8
Connections:
- J1 pad 10: /~{RESET} -> /~{RD}
- J1 pad 12: /~{RD} -> /~{WR}
- J1 pad 14: /~{WR} -> /R/~{W}
- J1 pad 16: /R/~{W} -> /~{CBLK}
- J1 pad 18: /USR1 -> /~{IORQ}
- J1 pad 20: /USR2 -> /~{MREQ}
- J1 pad 24: /~{MREQ} -> /BA
- J1 pad 26: /~{IORQ} -> /BS
- J1 pad 28: /~{CBLK} -> /USR1
- J1 pad 30: /~{BREQ} -> /USR2
- J1 pad 32: /~{HALT} -> /USR3
- J1 pad 34: /~{MRDY} -> /USR4
- J1 pad 36: /BA -> /~{BREQ}
- J1 pad 38: /BS -> /~{HALT}
- J1 pad 39: /~{MMU_{en}} -> /~{RESET}
- J1 pad 40: /~{RAM_{oe}} -> /~{MRDY}
- J1 pad 45: GND -> -12V
- J1 pad 46: GND -> +12V
- J1 pad 47: +12V -> GND
- J1 pad 48: /FIRQ1 -> GND
- J1 pad 49: -12V -> /~{RAM_{oe}}
- J1 pad 50: /FIRQ2 -> /FIRQ1
- J1 pad 51: GND -> /~{MMU_{en}}
- J1 pad 52: GND -> /FIRQ2
- J10 pad 10: /~{RESET} -> /~{RD}
- J10 pad 12: /~{RD} -> /~{WR}
- J10 pad 14: /~{WR} -> /R/~{W}
- J10 pad 16: /R/~{W} -> /~{CBLK}
- J10 pad 18: /USR1 -> /~{IORQ}
- J10 pad 20: /USR2 -> /~{MREQ}
- J10 pad 24: /~{MREQ} -> /BA
- J10 pad 26: /~{IORQ} -> /BS
- J10 pad 28: /~{CBLK} -> /USR1
- J10 pad 30: /~{BREQ} -> /USR2
- J10 pad 32: /~{HALT} -> /USR3
- J10 pad 34: /~{MRDY} -> /USR4
- J10 pad 36: /BA -> /~{BREQ}
- J10 pad 38: /BS -> /~{HALT}
- J10 pad 39: /~{MMU_{en}} -> /~{RESET}
- J10 pad 40: /~{RAM_{oe}} -> /~{MRDY}
- J10 pad 45: GND -> -12V
- J10 pad 46: GND -> +12V
- J10 pad 47: +12V -> GND
- J10 pad 48: /FIRQ1 -> GND
- J10 pad 49: -12V -> /~{RAM_{oe}}
- J10 pad 50: /FIRQ2 -> /FIRQ1
- J10 pad 51: GND -> /~{MMU_{en}}
- J10 pad 52: GND -> /FIRQ2
- J11 pad 10: /~{RESET} -> /~{RD}
- J11 pad 12: /~{RD} -> /~{WR}
- J11 pad 14: /~{WR} -> /R/~{W}
- J11 pad 16: /R/~{W} -> /~{CBLK}
- J11 pad 18: /USR1 -> /~{IORQ}
- J11 pad 20: /USR2 -> /~{MREQ}
- J11 pad 24: /~{MREQ} -> /BA
- J11 pad 26: /~{IORQ} -> /BS
- J11 pad 28: /~{CBLK} -> /USR1
- J11 pad 30: /~{BREQ} -> /USR2
- J11 pad 32: /~{HALT} -> /USR3
- J11 pad 34: /~{MRDY} -> /USR4
- J11 pad 36: /BA -> /~{BREQ}
- J11 pad 38: /BS -> /~{HALT}
- J11 pad 39: /~{MMU_{en}} -> /~{RESET}
- J11 pad 40: /~{RAM_{oe}} -> /~{MRDY}
- J11 pad 45: GND -> -12V
- J11 pad 46: GND -> +12V
- J11 pad 47: +12V -> GND
- J11 pad 48: /FIRQ1 -> GND
- J11 pad 49: -12V -> /~{RAM_{oe}}
- J11 pad 50: /FIRQ2 -> /FIRQ1
- J11 pad 51: GND -> /~{MMU_{en}}
- J11 pad 52: GND -> /FIRQ2
- J12 pad 10: /~{RESET} -> /~{RD}
- J12 pad 12: /~{RD} -> /~{WR}
- J12 pad 14: /~{WR} -> /R/~{W}
- J12 pad 16: /R/~{W} -> /~{CBLK}
- J12 pad 18: /USR1 -> /~{IORQ}
- J12 pad 20: /USR2 -> /~{MREQ}
- J12 pad 24: /~{MREQ} -> /BA
- J12 pad 26: /~{IORQ} -> /BS
- J12 pad 28: /~{CBLK} -> /USR1
- J12 pad 30: /~{BREQ} -> /USR2
- J12 pad 32: /~{HALT} -> /USR3
- J12 pad 34: /~{MRDY} -> /USR4
- J12 pad 36: /BA -> /~{BREQ}
- J12 pad 38: /BS -> /~{HALT}
- J12 pad 39: /~{MMU_{en}} -> /~{RESET}
- J12 pad 40: /~{RAM_{oe}} -> /~{MRDY}
- J12 pad 45: GND -> -12V
- J12 pad 46: GND -> +12V
- J12 pad 47: +12V -> GND
- J12 pad 48: /FIRQ1 -> GND
- J12 pad 49: -12V -> /~{RAM_{oe}}
- J12 pad 50: /FIRQ2 -> /FIRQ1
- J12 pad 51: GND -> /~{MMU_{en}}
- J12 pad 52: GND -> /FIRQ2
- J13 pad 10: /~{RESET} -> /~{RD}
- J13 pad 12: /~{RD} -> /~{WR}
- J13 pad 14: /~{WR} -> /R/~{W}
- J13 pad 16: /R/~{W} -> /~{CBLK}
- J13 pad 18: /USR1 -> /~{IORQ}
- J13 pad 20: /USR2 -> /~{MREQ}
- J13 pad 24: /~{MREQ} -> /BA
- J13 pad 26: /~{IORQ} -> /BS
- J13 pad 28: /~{CBLK} -> /USR1
- J13 pad 30: /~{BREQ} -> /USR2
- J13 pad 32: /~{HALT} -> /USR3
- J13 pad 34: /~{MRDY} -> /USR4
- J13 pad 36: /BA -> /~{BREQ}
- J13 pad 38: /BS -> /~{HALT}
- J13 pad 39: /~{MMU_{en}} -> /~{RESET}
- J13 pad 40: /~{RAM_{oe}} -> /~{MRDY}
- J13 pad 45: GND -> -12V
- J13 pad 46: GND -> +12V
- J13 pad 47: +12V -> GND
- J13 pad 48: /FIRQ1 -> GND
- J13 pad 49: -12V -> /~{RAM_{oe}}
- J13 pad 50: /FIRQ2 -> /FIRQ1
- J13 pad 51: GND -> /~{MMU_{en}}
- J13 pad 52: GND -> /FIRQ2
- J14 pad 10: /~{RESET} -> /~{RD}
- J14 pad 12: /~{RD} -> /~{WR}
- J14 pad 14: /~{WR} -> /R/~{W}
- J14 pad 16: /R/~{W} -> /~{CBLK}
- J14 pad 18: /USR1 -> /~{IORQ}
- J14 pad 20: /USR2 -> /~{MREQ}
- J14 pad 24: /~{MREQ} -> /BA
- J14 pad 26: /~{IORQ} -> /BS
- J14 pad 28: /~{CBLK} -> /USR1
- J14 pad 30: /~{BREQ} -> /USR2
- J14 pad 32: /~{HALT} -> /USR3
- J14 pad 34: /~{MRDY} -> /USR4
- J14 pad 36: /BA -> /~{BREQ}
- J14 pad 38: /BS -> /~{HALT}
- J14 pad 39: /~{MMU_{en}} -> /~{RESET}
- J14 pad 40: /~{RAM_{oe}} -> /~{MRDY}
- J14 pad 45: GND -> -12V
- J14 pad 46: GND -> +12V
- J14 pad 47: +12V -> GND
- J14 pad 48: /FIRQ1 -> GND
- J14 pad 49: -12V -> /~{RAM_{oe}}
- J14 pad 50: /FIRQ2 -> /FIRQ1
- J14 pad 51: GND -> /~{MMU_{en}}
- J14 pad 52: GND -> /FIRQ2
- J2 pad 10: /~{RESET} -> /~{RD}
- J2 pad 12: /~{RD} -> /~{WR}
- J2 pad 14: /~{WR} -> /R/~{W}
- J2 pad 16: /R/~{W} -> /~{CBLK}
- J2 pad 18: /USR1 -> /~{IORQ}
- J2 pad 20: /USR2 -> /~{MREQ}
- J2 pad 24: /~{MREQ} -> /BA
- J2 pad 26: /~{IORQ} -> /BS
- J2 pad 28: /~{CBLK} -> /USR1
- J2 pad 30: /~{BREQ} -> /USR2
- J2 pad 32: /~{HALT} -> /USR3
- J2 pad 34: /~{MRDY} -> /USR4
- J2 pad 36: /BA -> /~{BREQ}
- J2 pad 38: /BS -> /~{HALT}
- J2 pad 39: /~{MMU_{en}} -> /~{RESET}
- J2 pad 40: /~{RAM_{oe}} -> /~{MRDY}
- J2 pad 45: GND -> -12V
- J2 pad 46: GND -> +12V
- J2 pad 47: +12V -> GND
- J2 pad 48: /FIRQ1 -> GND
- J2 pad 49: -12V -> /~{RAM_{oe}}
- J2 pad 50: /FIRQ2 -> /FIRQ1
- J2 pad 51: GND -> /~{MMU_{en}}
- J2 pad 52: GND -> /FIRQ2
- J3 pad 10: /~{RESET} -> /~{RD}
- J3 pad 12: /~{RD} -> /~{WR}
- J3 pad 14: /~{WR} -> /R/~{W}
- J3 pad 16: /R/~{W} -> /~{CBLK}
- J3 pad 18: /USR1 -> /~{IORQ}
- J3 pad 20: /USR2 -> /~{MREQ}
- J3 pad 24: /~{MREQ} -> /BA
- J3 pad 26: /~{IORQ} -> /BS
- J3 pad 28: /~{CBLK} -> /USR1
- J3 pad 30: /~{BREQ} -> /USR2
- J3 pad 32: /~{HALT} -> /USR3
- J3 pad 34: /~{MRDY} -> /USR4
- J3 pad 36: /BA -> /~{BREQ}
- J3 pad 38: /BS -> /~{HALT}
- J3 pad 39: /~{MMU_{en}} -> /~{RESET}
- J3 pad 40: /~{RAM_{oe}} -> /~{MRDY}
- J3 pad 45: GND -> -12V
- J3 pad 46: GND -> +12V
- J3 pad 47: +12V -> GND
- J3 pad 48: /FIRQ1 -> GND
- J3 pad 49: -12V -> /~{RAM_{oe}}
- J3 pad 50: /FIRQ2 -> /FIRQ1
- J3 pad 51: GND -> /~{MMU_{en}}
- J3 pad 52: GND -> /FIRQ2
- J4 pad 10: /~{RESET} -> /~{RD}
- J4 pad 12: /~{RD} -> /~{WR}
- J4 pad 14: /~{WR} -> /R/~{W}
- J4 pad 16: /R/~{W} -> /~{CBLK}
- J4 pad 18: /USR1 -> /~{IORQ}
- J4 pad 20: /USR2 -> /~{MREQ}
- J4 pad 24: /~{MREQ} -> /BA
- J4 pad 26: /~{IORQ} -> /BS
- J4 pad 28: /~{CBLK} -> /USR1
- J4 pad 30: /~{BREQ} -> /USR2
- J4 pad 32: /~{HALT} -> /USR3
- J4 pad 34: /~{MRDY} -> /USR4
- J4 pad 36: /BA -> /~{BREQ}
- J4 pad 38: /BS -> /~{HALT}
- J4 pad 39: /~{MMU_{en}} -> /~{RESET}
- J4 pad 40: /~{RAM_{oe}} -> /~{MRDY}
- J4 pad 45: GND -> -12V
- J4 pad 46: GND -> +12V
- J4 pad 47: +12V -> GND
- J4 pad 48: /FIRQ1 -> GND
- J4 pad 49: -12V -> /~{RAM_{oe}}
- J4 pad 50: /FIRQ2 -> /FIRQ1
- J4 pad 51: GND -> /~{MMU_{en}}
- J4 pad 52: GND -> /FIRQ2
- J5 pad 10: /~{RESET} -> /~{RD}
- J5 pad 12: /~{RD} -> /~{WR}
- J5 pad 14: /~{WR} -> /R/~{W}
- J5 pad 16: /R/~{W} -> /~{CBLK}
- J5 pad 18: /USR1 -> /~{IORQ}
- J5 pad 20: /USR2 -> /~{MREQ}
- J5 pad 24: /~{MREQ} -> /BA
- J5 pad 26: /~{IORQ} -> /BS
- J5 pad 28: /~{CBLK} -> /USR1
- J5 pad 30: /~{BREQ} -> /USR2
- J5 pad 32: /~{HALT} -> /USR3
- J5 pad 34: /~{MRDY} -> /USR4
- J5 pad 36: /BA -> /~{BREQ}
- J5 pad 38: /BS -> /~{HALT}
- J5 pad 39: /~{MMU_{en}} -> /~{RESET}
- J5 pad 40: /~{RAM_{oe}} -> /~{MRDY}
- J5 pad 45: GND -> -12V
- J5 pad 46: GND -> +12V
- J5 pad 47: +12V -> GND
- J5 pad 48: /FIRQ1 -> GND
- J5 pad 49: -12V -> /~{RAM_{oe}}
- J5 pad 50: /FIRQ2 -> /FIRQ1
- J5 pad 51: GND -> /~{MMU_{en}}
- J5 pad 52: GND -> /FIRQ2
- J6 pad 10: /~{RESET} -> /~{RD}
- J6 pad 12: /~{RD} -> /~{WR}
- J6 pad 14: /~{WR} -> /R/~{W}
- J6 pad 16: /R/~{W} -> /~{CBLK}
- J6 pad 18: /USR1 -> /~{IORQ}
- J6 pad 20: /USR2 -> /~{MREQ}
- J6 pad 24: /~{MREQ} -> /BA
- J6 pad 26: /~{IORQ} -> /BS
- J6 pad 28: /~{CBLK} -> /USR1
- J6 pad 30: /~{BREQ} -> /USR2
- J6 pad 32: /~{HALT} -> /USR3
- J6 pad 34: /~{MRDY} -> /USR4
- J6 pad 36: /BA -> /~{BREQ}
- J6 pad 38: /BS -> /~{HALT}
- J6 pad 39: /~{MMU_{en}} -> /~{RESET}
- J6 pad 40: /~{RAM_{oe}} -> /~{MRDY}
- J6 pad 45: GND -> -12V
- J6 pad 46: GND -> +12V
- J6 pad 47: +12V -> GND
- J6 pad 48: /FIRQ1 -> GND
- J6 pad 49: -12V -> /~{RAM_{oe}}
- J6 pad 50: /FIRQ2 -> /FIRQ1
- J6 pad 51: GND -> /~{MMU_{en}}
- J6 pad 52: GND -> /FIRQ2
- J7 pad 1: unconnected-(J8-+3.3V-Pad1) -> +3V3
- J7 pad 13: unconnected-(J8-+3.3V-Pad13) -> +3V3
- J7 pad 2: unconnected-(J8-+3.3V-Pad2) -> +3V3
- J7 pad 21: unconnected-(J8-+5V-Pad21) -> +5V
- J7 pad 22: unconnected-(J8-+5V-Pad22) -> +5V
- J7 pad 4: +5V -> unconnected-(J7-+5V-Pad4)
- J8 pad 10: /~{RESET} -> /~{RD}
- J8 pad 12: /~{RD} -> /~{WR}
- J8 pad 14: /~{WR} -> /R/~{W}
- J8 pad 16: /R/~{W} -> /~{CBLK}
- J8 pad 18: /USR1 -> /~{IORQ}
- J8 pad 20: /USR2 -> /~{MREQ}
- J8 pad 24: /~{MREQ} -> /BA
- J8 pad 26: /~{IORQ} -> /BS
- J8 pad 28: /~{CBLK} -> /USR1
- J8 pad 30: /~{BREQ} -> /USR2
- J8 pad 32: /~{HALT} -> /USR3
- J8 pad 34: /~{MRDY} -> /USR4
- J8 pad 36: /BA -> /~{BREQ}
- J8 pad 38: /BS -> /~{HALT}
- J8 pad 39: /~{MMU_{en}} -> /~{RESET}
- J8 pad 40: /~{RAM_{oe}} -> /~{MRDY}
- J8 pad 45: GND -> -12V
- J8 pad 46: GND -> +12V
- J8 pad 47: +12V -> GND
- J8 pad 48: /FIRQ1 -> GND
- J8 pad 49: -12V -> /~{RAM_{oe}}
- J8 pad 50: /FIRQ2 -> /FIRQ1
- J8 pad 51: GND -> /~{MMU_{en}}
- J8 pad 52: GND -> /FIRQ2
- J9 pad 10: /~{RESET} -> /~{RD}
- J9 pad 12: /~{RD} -> /~{WR}
- J9 pad 14: /~{WR} -> /R/~{W}
- J9 pad 16: /R/~{W} -> /~{CBLK}
- J9 pad 18: /USR1 -> /~{IORQ}
- J9 pad 20: /USR2 -> /~{MREQ}
- J9 pad 24: /~{MREQ} -> /BA
- J9 pad 26: /~{IORQ} -> /BS
- J9 pad 28: /~{CBLK} -> /USR1
- J9 pad 30: /~{BREQ} -> /USR2
- J9 pad 32: /~{HALT} -> /USR3
- J9 pad 34: /~{MRDY} -> /USR4
- J9 pad 36: /BA -> /~{BREQ}
- J9 pad 38: /BS -> /~{HALT}
- J9 pad 39: /~{MMU_{en}} -> /~{RESET}
- J9 pad 40: /~{RAM_{oe}} -> /~{MRDY}
- J9 pad 45: GND -> -12V
- J9 pad 46: GND -> +12V
- J9 pad 47: +12V -> GND
- J9 pad 48: /FIRQ1 -> GND
- J9 pad 49: -12V -> /~{RAM_{oe}}
- J9 pad 50: /FIRQ2 -> /FIRQ1
- J9 pad 51: GND -> /~{MMU_{en}}
- J9 pad 52: GND -> /FIRQ2
Routing:
- net GND: track 1469.3 -> 1898.2 mm
- net /USR3: track 0.00 -> 259.6 mm
- net /USR4: track 0.00 -> 259.6 mm
- net +3V3: track 244.9 -> 473.4 mm, vias 0 -> 1
- net +5V: track 0.00 -> 226.6 mm
- net +12V: track 236.8 -> 385.7 mm, vias 0 -> 1
- net -12V: track 236.8 -> 385.0 mm, vias 0 -> 1
- net /~{RAM_{oe}}: track 252.7 -> 262.0 mm
- net /~{RESET}: track 252.7 -> 262.0 mm
- net /~{HALT}: track 252.7 -> 259.6 mm
- net /FIRQ2: track 252.7 -> 259.6 mm
- net /BA: track 252.7 -> 259.6 mm
- net /~{CBLK}: track 252.7 -> 259.6 mm
- net /~{IORQ}: track 252.7 -> 259.6 mm
- net /~{BREQ}: track 252.7 -> 259.6 mm
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- added copper zone on In1.Cu, net +5V
- added copper zone on In2.Cu, net GND
Other:
- board size 285.8 x 124.5 mm -> 297.2 x 124.5 mm
- board text added: "72-PIN CARD EDGE PASSIVE BACKPLANE"
- board text removed: "16-BIT ISA PASSIVE ATX BACKPLANE"
