File: Episode4/Episode4.kicad_sch (KiCad schematic)
At the start: 41 parts, among them J1 CARD, J10 CARD, J11 CARD, J12 CARD, J13 CARD, J14 CARD, J2 CARD, J3 CARD, J4 CARD, J5 CARD, J6 CARD, J7 BB Con, J8 ATX POWER, J9 CARD, SW1 POWER, U1 74HCT14, U2 74HCT74

Commit message: Reworked bus line order, capacitor and trace placement
Parts:
- removed D1: TVS 5V, Diode_SMD:D_SMB, symbol Diode:SM6T6V8A
- removed D2: TVS 3V3, Diode_SMD:D_SMB, symbol Diode:SM6T6V8A
- removed D3, D4: TVS 12V, Diode_SMD:D_SMB, symbol Diode:SM6T6V8A
- added D5: TVS 5V, Diode_SMD:D_SMB, symbol Diode:SM6T6V8A
- renumbered D5 to D1, D6 to D2, D7 to D3, D8 to D4, J8 to J7, J7 to J8
Connections:
- net +12V: now also J1.46 (B23), J10.46 (B23), J11.46 (B23), J12.46 (B23), J13.46 (B23), J14.46 (B23), J2.46 (B23), J3.46 (B23), J4.46 (B23), J5.46 (B23), J6.46 (B23), J8.46 (Pin_46), J9.46 (B23); no longer J1.47 (A24), J10.47 (A24), J11.47 (A24), J12.47 (A24), J13.47 (A24), J14.47 (A24), J2.47 (A24), J3.47 (A24), J4.47 (A24), J5.47 (A24), J6.47 (A24), J8.47 (Pin_47), J9.47 (A24)
- net +3V3: now also J7.1 (+3.3V), J7.13 (+3.3V), J7.2 (+3.3V)
- net +5V: now also J7.21 (+5V), J7.22 (+5V), D5.1 (A1); no longer J7.4 (+5V)
- net -12V: now also J1.45 (A23), J10.45 (A23), J11.45 (A23), J12.45 (A23), J13.45 (A23), J14.45 (A23), J2.45 (A23), J3.45 (A23), J4.45 (A23), J5.45 (A23), J6.45 (A23), J8.45 (Pin_45), J9.45 (A23); no longer J1.49 (A25), J10.49 (A25), J11.49 (A25), J12.49 (A25), J13.49 (A25), J14.49 (A25), J2.49 (A25), J3.49 (A25), J4.49 (A25), J5.49 (A25), J6.49 (A25), J8.49 (Pin_49), J9.49 (A25)
- net BA: now also J1.24 (B12), J10.24 (B12), J11.24 (B12), J12.24 (B12), J13.24 (B12), J14.24 (B12), J2.24 (B12), J3.24 (B12), J4.24 (B12), J5.24 (B12), J6.24 (B12), J8.24 (Pin_24), J9.24 (B12); no longer J1.36 (B18), J10.36 (B18), J11.36 (B18), J12.36 (B18), J13.36 (B18), J14.36 (B18), J2.36 (B18), J3.36 (B18), J4.36 (B18), J5.36 (B18), J6.36 (B18), J8.36 (Pin_36), J9.36 (B18)
- net BS: now also J1.26 (B13), J10.26 (B13), J11.26 (B13), J12.26 (B13), J13.26 (B13), J14.26 (B13), J2.26 (B13), J3.26 (B13), J4.26 (B13), J5.26 (B13), J6.26 (B13), J8.26 (Pin_26), J9.26 (B13); no longer J1.38 (B19), J10.38 (B19), J11.38 (B19), J12.38 (B19), J13.38 (B19), J14.38 (B19), J2.38 (B19), J3.38 (B19), J4.38 (B19), J5.38 (B19), J6.38 (B19), J8.38 (Pin_38), J9.38 (B19)
- net FIRQ1: now also J1.50 (B25), J10.50 (B25), J11.50 (B25), J12.50 (B25), J13.50 (B25), J14.50 (B25), J2.50 (B25), J3.50 (B25), J4.50 (B25), J5.50 (B25), J6.50 (B25), J8.50 (Pin_50), J9.50 (B25); no longer J1.48 (B24), J10.48 (B24), J11.48 (B24), J12.48 (B24), J13.48 (B24), J14.48 (B24), J2.48 (B24), J3.48 (B24), J4.48 (B24), J5.48 (B24), J6.48 (B24), J8.48 (Pin_48), J9.48 (B24)
- net FIRQ2: now also J1.52 (B26), J10.52 (B26), J11.52 (B26), J12.52 (B26), J13.52 (B26), J14.52 (B26), J2.52 (B26), J3.52 (B26), J4.52 (B26), J5.52 (B26), J6.52 (B26), J8.52 (Pin_52), J9.52 (B26); no longer J1.50 (B25), J10.50 (B25), J11.50 (B25), J12.50 (B25), J13.50 (B25), J14.50 (B25), J2.50 (B25), J3.50 (B25), J4.50 (B25), J5.50 (B25), J6.50 (B25), J8.50 (Pin_50), J9.50 (B25)
- net GND: now also J1.47 (A24), J1.48 (B24), J10.47 (A24), J10.48 (B24), J11.47 (A24), J11.48 (B24), J12.47 (A24), J12.48 (B24), J13.47 (A24), J13.48 (B24), J14.47 (A24), J14.48 (B24), J2.47 (A24), J2.48 (B24), J3.47 (A24), J3.48 (B24), J4.47 (A24), J4.48 (B24), J5.47 (A24), J5.48 (B24), J6.47 (A24), J6.48 (B24), J8.47 (Pin_47), J8.48 (Pin_48), J9.47 (A24), J9.48 (B24), D5.2 (A2); no longer J1.45 (A23), J1.46 (B23), J1.51 (A26), J1.52 (B26), J10.45 (A23), J10.46 (B23), J10.51 (A26), J10.52 (B26), J11.45 (A23), J11.46 (B23), J11.51 (A26), J11.52 (B26), J12.45 (A23), J12.46 (B23), J12.51 (A26), J12.52 (B26), J13.45 (A23), J13.46 (B23), J13.51 (A26), J13.52 (B26), J14.45 (A23), J14.46 (B23), J14.51 (A26), J14.52 (B26), J2.45 (A23), J2.46 (B23), J2.51 (A26), J2.52 (B26), J3.45 (A23), J3.46 (B23), J3.51 (A26), J3.52 (B26), J4.45 (A23), J4.46 (B23), J4.51 (A26), J4.52 (B26), J5.45 (A23), J5.46 (B23), J5.51 (A26), J5.52 (B26), J6.45 (A23), J6.46 (B23), J6.51 (A26), J6.52 (B26), J8.45 (Pin_45), J8.46 (Pin_46), J8.51 (Pin_51), J8.52 (Pin_52), J9.45 (A23), J9.46 (B23), J9.51 (A26), J9.52 (B26)
- net R/~{W}: now also J1.14 (B7), J10.14 (B7), J11.14 (B7), J12.14 (B7), J13.14 (B7), J14.14 (B7), J2.14 (B7), J3.14 (B7), J4.14 (B7), J5.14 (B7), J6.14 (B7), J8.14 (Pin_14), J9.14 (B7); no longer J1.16 (B8), J10.16 (B8), J11.16 (B8), J12.16 (B8), J13.16 (B8), J14.16 (B8), J2.16 (B8), J3.16 (B8), J4.16 (B8), J5.16 (B8), J6.16 (B8), J8.16 (Pin_16), J9.16 (B8)
- net USR1: now also J1.28 (B14), J10.28 (B14), J11.28 (B14), J12.28 (B14), J13.28 (B14), J14.28 (B14), J2.28 (B14), J3.28 (B14), J4.28 (B14), J5.28 (B14), J6.28 (B14), J8.28 (Pin_28), J9.28 (B14); no longer J1.18 (B9), J10.18 (B9), J11.18 (B9), J12.18 (B9), J13.18 (B9), J14.18 (B9), J2.18 (B9), J3.18 (B9), J4.18 (B9), J5.18 (B9), J6.18 (B9), J8.18 (Pin_18), J9.18 (B9)
- net USR2: now also J1.30 (B15), J10.30 (B15), J11.30 (B15), J12.30 (B15), J13.30 (B15), J14.30 (B15), J2.30 (B15), J3.30 (B15), J4.30 (B15), J5.30 (B15), J6.30 (B15), J8.30 (Pin_30), J9.30 (B15); no longer J1.20 (B10), J10.20 (B10), J11.20 (B10), J12.20 (B10), J13.20 (B10), J14.20 (B10), J2.20 (B10), J3.20 (B10), J4.20 (B10), J5.20 (B10), J6.20 (B10), J8.20 (Pin_20), J9.20 (B10)
- net ~{BREQ}: now also J1.36 (B18), J10.36 (B18), J11.36 (B18), J12.36 (B18), J13.36 (B18), J14.36 (B18), J2.36 (B18), J3.36 (B18), J4.36 (B18), J5.36 (B18), J6.36 (B18), J8.36 (Pin_36), J9.36 (B18); no longer J1.30 (B15), J10.30 (B15), J11.30 (B15), J12.30 (B15), J13.30 (B15), J14.30 (B15), J2.30 (B15), J3.30 (B15), J4.30 (B15), J5.30 (B15), J6.30 (B15), J8.30 (Pin_30), J9.30 (B15)
- net ~{CBLK}: now also J1.16 (B8), J10.16 (B8), J11.16 (B8), J12.16 (B8), J13.16 (B8), J14.16 (B8), J2.16 (B8), J3.16 (B8), J4.16 (B8), J5.16 (B8), J6.16 (B8), J8.16 (Pin_16), J9.16 (B8); no longer J1.28 (B14), J10.28 (B14), J11.28 (B14), J12.28 (B14), J13.28 (B14), J14.28 (B14), J2.28 (B14), J3.28 (B14), J4.28 (B14), J5.28 (B14), J6.28 (B14), J8.28 (Pin_28), J9.28 (B14)
- net ~{HALT}: now also J1.38 (B19), J10.38 (B19), J11.38 (B19), J12.38 (B19), J13.38 (B19), J14.38 (B19), J2.38 (B19), J3.38 (B19), J4.38 (B19), J5.38 (B19), J6.38 (B19), J8.38 (Pin_38), J9.38 (B19); no longer J1.32 (B16), J10.32 (B16), J11.32 (B16), J12.32 (B16), J13.32 (B16), J14.32 (B16), J2.32 (B16), J3.32 (B16), J4.32 (B16), J5.32 (B16), J6.32 (B16), J8.32 (Pin_32), J9.32 (B16)
- net ~{IORQ}: now also J1.18 (B9), J10.18 (B9), J11.18 (B9), J12.18 (B9), J13.18 (B9), J14.18 (B9), J2.18 (B9), J3.18 (B9), J4.18 (B9), J5.18 (B9), J6.18 (B9), J8.18 (Pin_18), J9.18 (B9); no longer J1.26 (B13), J10.26 (B13), J11.26 (B13), J12.26 (B13), J13.26 (B13), J14.26 (B13), J2.26 (B13), J3.26 (B13), J4.26 (B13), J5.26 (B13), J6.26 (B13), J8.26 (Pin_26), J9.26 (B13)
- net ~{MMU_{en}}: now also J1.51 (A26), J10.51 (A26), J11.51 (A26), J12.51 (A26), J13.51 (A26), J14.51 (A26), J2.51 (A26), J3.51 (A26), J4.51 (A26), J5.51 (A26), J6.51 (A26), J8.51 (Pin_51), J9.51 (A26); no longer J1.39 (A20), J10.39 (A20), J11.39 (A20), J12.39 (A20), J13.39 (A20), J14.39 (A20), J2.39 (A20), J3.39 (A20), J4.39 (A20), J5.39 (A20), J6.39 (A20), J8.39 (Pin_39), J9.39 (A20)
- net ~{MRDY}: now also J1.40 (B20), J10.40 (B20), J11.40 (B20), J12.40 (B20), J13.40 (B20), J14.40 (B20), J2.40 (B20), J3.40 (B20), J4.40 (B20), J5.40 (B20), J6.40 (B20), J8.40 (Pin_40), J9.40 (B20); no longer J1.34 (B17), J10.34 (B17), J11.34 (B17), J12.34 (B17), J13.34 (B17), J14.34 (B17), J2.34 (B17), J3.34 (B17), J4.34 (B17), J5.34 (B17), J6.34 (B17), J8.34 (Pin_34), J9.34 (B17)
- net ~{MREQ}: now also J1.20 (B10), J10.20 (B10), J11.20 (B10), J12.20 (B10), J13.20 (B10), J14.20 (B10), J2.20 (B10), J3.20 (B10), J4.20 (B10), J5.20 (B10), J6.20 (B10), J8.20 (Pin_20), J9.20 (B10); no longer J1.24 (B12), J10.24 (B12), J11.24 (B12), J12.24 (B12), J13.24 (B12), J14.24 (B12), J2.24 (B12), J3.24 (B12), J4.24 (B12), J5.24 (B12), J6.24 (B12), J8.24 (Pin_24), J9.24 (B12)
- net ~{RAM_{oe}}: now also J1.49 (A25), J10.49 (A25), J11.49 (A25), J12.49 (A25), J13.49 (A25), J14.49 (A25), J2.49 (A25), J3.49 (A25), J4.49 (A25), J5.49 (A25), J6.49 (A25), J8.49 (Pin_49), J9.49 (A25); no longer J1.40 (B20), J10.40 (B20), J11.40 (B20), J12.40 (B20), J13.40 (B20), J14.40 (B20), J2.40 (B20), J3.40 (B20), J4.40 (B20), J5.40 (B20), J6.40 (B20), J8.40 (Pin_40), J9.40 (B20)
- net ~{RD}: now also J1.10 (B5), J10.10 (B5), J11.10 (B5), J12.10 (B5), J13.10 (B5), J14.10 (B5), J2.10 (B5), J3.10 (B5), J4.10 (B5), J5.10 (B5), J6.10 (B5), J8.10 (Pin_10), J9.10 (B5); no longer J1.12 (B6), J10.12 (B6), J11.12 (B6), J12.12 (B6), J13.12 (B6), J14.12 (B6), J2.12 (B6), J3.12 (B6), J4.12 (B6), J5.12 (B6), J6.12 (B6), J8.12 (Pin_12), J9.12 (B6)
- net ~{RESET}: now also J1.39 (A20), J10.39 (A20), J11.39 (A20), J12.39 (A20), J13.39 (A20), J14.39 (A20), J2.39 (A20), J3.39 (A20), J4.39 (A20), J5.39 (A20), J6.39 (A20), J8.39 (Pin_39), J9.39 (A20); no longer J1.10 (B5), J10.10 (B5), J11.10 (B5), J12.10 (B5), J13.10 (B5), J14.10 (B5), J2.10 (B5), J3.10 (B5), J4.10 (B5), J5.10 (B5), J6.10 (B5), J8.10 (Pin_10), J9.10 (B5)
- net ~{WR}: now also J1.12 (B6), J10.12 (B6), J11.12 (B6), J12.12 (B6), J13.12 (B6), J14.12 (B6), J2.12 (B6), J3.12 (B6), J4.12 (B6), J5.12 (B6), J6.12 (B6), J8.12 (Pin_12), J9.12 (B6); no longer J1.14 (B7), J10.14 (B7), J11.14 (B7), J12.14 (B7), J13.14 (B7), J14.14 (B7), J2.14 (B7), J3.14 (B7), J4.14 (B7), J5.14 (B7), J6.14 (B7), J8.14 (Pin_14), J9.14 (B7)
- new net USR3: J1.32 (B16), J10.32 (B16), J11.32 (B16), J12.32 (B16), J13.32 (B16), J14.32 (B16), J2.32 (B16), J3.32 (B16), J4.32 (B16), J5.32 (B16), J6.32 (B16), J8.32 (Pin_32), J9.32 (B16)
- new net USR4: J1.34 (B17), J10.34 (B17), J11.34 (B17), J12.34 (B17), J13.34 (B17), J14.34 (B17), J2.34 (B17), J3.34 (B17), J4.34 (B17), J5.34 (B17), J6.34 (B17), J8.34 (Pin_34), J9.34 (B17)
- no-connect marks 13 -> 9
Other:
- note added: "ESD Protection"
- note removed: "ESD Protection (At ATX PSU connector level)"
- note removed: "ESD Protection (At header pin connector level)"
- moved on the sheet: C1, C2, D1, D2, D3, D4, J7, R1, R2, R3, R4, SW1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
