File: Episode5 - CPU card/CPU_RESET_BUFFERS.kicad_sch (KiCad schematic)
At the start: 41 parts, among them SW1 RESET, SW2 NMI, U1 74AHCT541, U2 74AHCT245, U3 HD63C09P, U4 74AHCT541, U5 74AHCT244, U6 ATF22V10C, U7 ATF22V10C, U8 MIC1232, X1 X MHz

Commit message: Toyed with CPU PCB
Parts:
- removed R1, R2, R3, R4, R5, R6, R7, R8: 4K7Ω, symbol Device:R_Small_US
- added RN3: 4K7Ω, Resistor_THT:R_Array_SIP9, symbol Device:R_Network08_US
- C10: renamed from C12; footprint (none) -> Capacitor_THT:C_Disc_D3.0mm_W1.6mm_P2.50mm
- C2, C3, C4, C5, C6, C7, C8: footprint (none) -> Capacitor_THT:C_Disc_D3.0mm_W1.6mm_P2.50mm
- C9: renamed from C11; footprint (none) -> Capacitor_THT:C_Disc_D3.0mm_W1.6mm_P2.50mm
- D1: footprint (none) -> LED_THT:LED_D5.0mm
- R1: renamed from R9; footprint (none) -> Resistor_THT:R_Axial_DIN0207_L6.3mm_D2.5mm_P10.16mm_Horizontal
- R2: renamed from R10; footprint (none) -> Resistor_THT:R_Axial_DIN0207_L6.3mm_D2.5mm_P10.16mm_Horizontal
- R3: renamed from R11; footprint (none) -> Resistor_THT:R_Axial_DIN0207_L6.3mm_D2.5mm_P10.16mm_Horizontal
- R4: renamed from R12; footprint (none) -> Resistor_THT:R_Axial_DIN0207_L6.3mm_D2.5mm_P10.16mm_Horizontal
- R5: renamed from R13; footprint (none) -> Resistor_THT:R_Axial_DIN0207_L6.3mm_D2.5mm_P10.16mm_Horizontal
- R7: renamed from R15; footprint (none) -> Resistor_THT:R_Axial_DIN0207_L6.3mm_D2.5mm_P10.16mm_Horizontal
- RN1, RN2: footprint Package_DIP:DIP-16_W7.62mm -> Package_DIP:DIP-16_W7.62mm_Socket
- RN4: renamed from RN3; footprint Package_DIP:DIP-16_W7.62mm -> Package_DIP:DIP-16_W7.62mm_Socket
- SW1, SW2: footprint (none) -> Button_Switch_THT:SW_Tactile_SKHH_Angled
- U1, U4: value 74AHCT541 -> 74AHCT244; symbol 74xx:74HCT541 -> 74xx:74AHCT244
- U5: footprint (none) -> Package_DIP:DIP-20_W7.62mm_Socket
- U6, U7: footprint Package_DIP:DIP-24_W7.62mm_Socket_LongPads -> Package_DIP:DIP-24_W7.62mm_Socket
- renumbered R14 to R6, R16 to R8
Connections:
- net +5V: now also RN3.1 (common)
- net A0: now also RN1.8 (R8.1); no longer RN1.16 (R1.2)
- net A1: now also RN1.7 (R7.1); no longer RN1.15 (R2.2)
- net A10: now also RN4.6 (R6.1); no longer RN4.14 (R3.2)
- net A11: now also RN4.5 (R5.1); no longer RN4.13 (R4.2)
- net A12: now also RN4.4 (R4.1); no longer RN4.12 (R5.2)
- net A13: now also RN4.3 (R3.1); no longer RN4.11 (R6.2)
- net A14: now also RN4.2 (R2.1); no longer RN4.10 (R7.2)
- net A15: now also RN4.1 (R1.1); no longer RN4.9 (R8.2)
- net A2: now also RN1.6 (R6.1); no longer RN1.14 (R3.2)
- net A3: now also RN1.5 (R5.1); no longer RN1.13 (R4.2)
- net A4: now also RN1.4 (R4.1); no longer RN1.12 (R5.2)
- net A5: now also RN1.3 (R3.1); no longer RN1.11 (R6.2)
- net A6: now also RN1.2 (R2.1); no longer RN1.10 (R7.2)
- net A7: now also RN1.1 (R1.1); no longer RN1.9 (R8.2)
- net A8: now also RN4.8 (R8.1); no longer RN4.16 (R1.2)
- net A9: now also RN4.7 (R7.1); no longer RN4.15 (R2.2)
- net AA1: now also U1.4 (1A1); no longer U1.3 (A1)
- net AA10: now also U4.6 (1A2); no longer U4.4 (A2)
- net AA11: now also U4.8 (1A3); no longer U4.5 (A3)
- net AA12: now also U4.17 (2A0); no longer U4.6 (A4)
- net AA13: now also U4.15 (2A1); no longer U4.7 (A5)
- net AA14: now also U4.13 (2A2); no longer U4.8 (A6)
- net AA15: now also U4.11 (2A3); no longer U4.9 (A7)
- net AA2: now also U1.6 (1A2); no longer U1.4 (A2)
- net AA3: now also U1.8 (1A3); no longer U1.5 (A3)
- net AA4: now also U1.17 (2A0); no longer U1.6 (A4)
- net AA5: now also U1.15 (2A1); no longer U1.7 (A5)
- net AA6: now also U1.13 (2A2); no longer U1.8 (A6)
- net AA7: now also U1.11 (2A3); no longer U1.9 (A7)
- net AA9: now also U4.4 (1A1); no longer U4.3 (A1)
- net D0: now also RN2.8 (R8.1); no longer RN2.16 (R1.2)
- net D1: now also RN2.7 (R7.1); no longer RN2.15 (R2.2)
- net D2: now also RN2.6 (R6.1); no longer RN2.14 (R3.2)
- net D3: now also RN2.5 (R5.1); no longer RN2.13 (R4.2)
- net D4: now also RN2.4 (R4.1); no longer RN2.12 (R5.2)
- net D5: now also RN2.3 (R3.1); no longer RN2.11 (R6.2)
- net D6: now also RN2.2 (R2.1); no longer RN2.10 (R7.2)
- net D7: now also RN2.1 (R1.1); no longer RN2.9 (R8.2)
- net GND: no longer U1.19 (G2), U4.19 (G2)
- net _{ub}BA: now also U1.19 (2OE), U4.19 (2OE)
- net ~{BREQ}: now also RN3.8 (R7)
- net ~{CART_{det}}: now also RN3.2 (R1)
- net ~{FIRQ}: now also RN3.5 (R4)
- net ~{HALT}: now also RN3.7 (R6)
- net ~{IRQ}: now also RN3.4 (R3)
- net ~{MRDY}: now also RN3.6 (R5)
- net ~{NMI}: now also RN3.3 (R2)
- net ~{RESET}: now also RN3.9 (R8)
- net at U2.2 (A0): now also RN2.9 (R8.2); no longer RN2.1 (R1.1)
- net at U2.3 (A1): now also RN2.10 (R7.2); no longer RN2.2 (R2.1)
- net at U2.4 (A2): now also RN2.11 (R6.2); no longer RN2.3 (R3.1)
- net at U2.5 (A3): now also RN2.12 (R5.2); no longer RN2.4 (R4.1)
- net at U2.6 (A4): now also RN2.13 (R4.2); no longer RN2.5 (R5.1)
- net at U2.7 (A5): now also RN2.14 (R3.2); no longer RN2.6 (R6.1)
- net at U2.8 (A6): now also RN2.15 (R2.2); no longer RN2.7 (R7.1)
- net at U2.9 (A7): now also RN2.16 (R1.2); no longer RN2.8 (R8.1)
- net at U1.18 (1Y0): now also RN1.9 (R8.2); no longer RN1.1 (R1.1)
- net at U1.16 (1Y1): now also RN1.10 (R7.2); no longer RN1.3 (R3.1)
- net at U1.14 (1Y2): now also RN1.11 (R6.2); no longer RN1.5 (R5.1)
- net at U1.12 (1Y3): now also RN1.12 (R5.2); no longer RN1.7 (R7.1)
- net at U4.12 (1Y3): now also RN4.12 (R5.2); no longer RN4.7 (R7.1)
- net at U4.14 (1Y2): now also RN4.11 (R6.2); no longer RN4.5 (R5.1)
- net at U4.16 (1Y1): now also RN4.10 (R7.2); no longer RN4.3 (R3.1)
- net at U4.18 (1Y0): now also RN4.9 (R8.2); no longer RN4.1 (R1.1)
- new net: RN1.13 (R4.2), U1.3 (2Y0)
- new net: RN1.14 (R3.2), U1.5 (2Y1)
- new net: RN1.15 (R2.2), U1.7 (2Y2)
- new net: RN1.16 (R1.2), U1.9 (2Y3)
- new net: RN4.13 (R4.2), U4.3 (2Y0)
- new net: RN4.14 (R3.2), U4.5 (2Y1)
- new net: RN4.15 (R2.2), U4.7 (2Y2)
- new net: RN4.16 (R1.2), U4.9 (2Y3)
Other:
- moved on the sheet: RN1, RN2, RN4
