File: Episode5 - CPU card/ROMRAM.kicad_sch (KiCad schematic)
At the start: 5 parts, among them U10 AS6C1008, U9 SST39SF010

Commit message: Toyed with CPU PCB
Parts:
- C11: renamed from C9; footprint (none) -> Capacitor_THT:C_Disc_D3.0mm_W1.6mm_P2.50mm
- C12: renamed from C10; footprint (none) -> Capacitor_THT:C_Disc_D3.0mm_W1.6mm_P2.50mm
- R9: renamed from R17; footprint (none) -> Resistor_THT:R_Axial_DIN0207_L6.3mm_D2.5mm_P10.16mm_Horizontal
- U10: footprint Package_DIP:DIP-32_W15.24mm -> Package_DIP:DIP-32_W15.24mm_Socket
- U9: footprint Package_DIP:DIP-32_W15.24mm -> Socket:DIP_Socket-32_W11.9mm_W12.7mm_W15.24mm_W17.78mm_W18.5mm_3M_232-1285-00-0602J
Changed lines of the file:
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@@
 		(on_board yes)
 		(dnp no)
-		(property "Reference" "R17"
+		(property "Reference" "R9"
 			(at 199.39 104.14 0)
 			(effects
@@
 			)
 		)
-		(property "Footprint" ""
+		(property "Footprint" "Resistor_THT:R_Axial_DIN0207_L6.3mm_D2.5mm_P10.16mm_Horizontal"
 			(at 196.85 105.41 0)
 			(effects
@@
 			(project "Episode5"
 				(path "/29787633-5c1f-4e4e-91db-ab6870e032bc/0ceebdfb-4953-4f6c-a4a7-697b591b5d1a"
-					(reference "R17")
+					(reference "R9")
 					(unit 1)
 				)
@@
 		(on_board yes)
 		(dnp no)
-		(property "Reference" "C9"
+		(property "Reference" "C11"
 			(at 15.875 193.04 0)
 			(effects
@@
 			)
 		)
-		(property "Footprint" ""
+		(property "Footprint" "Capacitor_THT:C_Disc_D3.0mm_W1.6mm_P2.50mm"
 			(at 13.97 194.31 0)
 			(effects
@@
 			(project "Episode5"
 				(path "/29787633-5c1f-4e4e-91db-ab6870e032bc/0ceebdfb-4953-4f6c-a4a7-697b591b5d1a"
-					(reference "C9")
+					(reference "C11")
 					(unit 1)
 				)
@@
 			)
 		)
-		(property "Footprint" "Package_DIP:DIP-32_W15.24mm"
+		(property "Footprint" "Socket:DIP_Socket-32_W11.9mm_W12.7mm_W15.24mm_W17.78mm_W18.5mm_3M_232-1285-00-0602J"
 			(at 114.3 100.33 0)
 			(effects
@@
 		(on_board yes)
 		(dnp no)
-		(property "Reference" "C10"
+		(property "Reference" "C12"
 			(at 26.035 193.04 0)
 			(effects
@@
 			)
 		)
-		(property "Footprint" ""
+		(property "Footprint" "Capacitor_THT:C_Disc_D3.0mm_W1.6mm_P2.50mm"
 			(at 24.13 194.31 0)
 			(effects
@@
 			(project "Episode5"
 				(path "/29787633-5c1f-4e4e-91db-ab6870e032bc/0ceebdfb-4953-4f6c-a4a7-697b591b5d1a"
-					(reference "C10")
+					(reference "C12")
 					(unit 1)
 				)
@@
 			)
 		)
-		(property "Footprint" "Package_DIP:DIP-32_W15.24mm"
+		(property "Footprint" "Package_DIP:DIP-32_W15.24mm_Socket"
 			(at 167.64 100.33 0)
 			(effects
